File: kicad/projects/CacheModule/CacheModule.kicad_pcb (KiCad board)
At the start: 2 copper layers, 118.1 x 12.7 mm, 20 parts, among them U1 CY7C1041D, U2 CY7C1041D, U3 CY7C1041D, U4 CY7C1041D, U5 CY7C1041D, U6 24LC00

Commit message: Some Updates
Parts:
- added C12: 100u, Capacitor_SMD:C_0603_1608Metric_Pad1.08x0.95mm_HandSolder, B.Cu at (144.7, 89.5)
- added C13: 100u, Capacitor_SMD:C_0603_1608Metric_Pad1.08x0.95mm_HandSolder, B.Cu at (148.1, 89.5)
- added C14: 100u, Capacitor_SMD:C_0603_1608Metric_Pad1.08x0.95mm_HandSolder, B.Cu at (159.3, 89.5)
- added C15: 100u, Capacitor_SMD:C_0603_1608Metric_Pad1.08x0.95mm_HandSolder, B.Cu at (163.6, 86.7)
- added C16: 100u, Capacitor_SMD:C_0603_1608Metric_Pad1.08x0.95mm_HandSolder, B.Cu at (163.5, 94.9)
- added U7: CY7C1041D, Package_SO:TSOP-II-44_10.16x18.41mm_P0.8mm, F.Cu at (124.5, 89.3)
- added U8: CY7C1041D, Package_SO:TSOP-II-44_10.16x18.41mm_P0.8mm, F.Cu at (95.3, 89.3)
- added U9: CY7C1041D, Package_SO:TSOP-II-44_10.16x18.41mm_P0.8mm, F.Cu at (139.1, 89.3)
- C9: moved to B.Cu
- J1: footprint m68k-hbc-conn:SIMM80_Cache_CardEdge -> m68k-hbc-conn:SIMM80_CardEdge
- TP1: footprint Connector_PinHeader_1.27mm:PinHeader_1x02_P1.27mm_Vertical -> Resistor_SMD:R_0402_1005Metric
- U1: value CY7C1041D -> 74LVC1G139; footprint Package_SO:TSOP-II-44_10.16x18.41mm_P0.8mm -> Package_SO:SSOP-8_3.9x5.05mm_P1.27mm
- U5: value CY7C1041D -> 24LC00; footprint Package_SO:TSOP-II-44_10.16x18.41mm_P0.8mm -> Package_SO:SOIC-8_3.9x4.9mm_P1.27mm
- U6: value 24LC00 -> CY7C1041D; footprint Package_SO:SOIC-8_3.9x4.9mm_P1.27mm -> Package_SO:TSOP-II-44_10.16x18.41mm_P0.8mm
- moved U1 93.8 mm to (163.6, 86.7), turned to 90 degrees
- moved U4 68.6 mm to (153.7, 89.3)
- moved U6 50.6 mm to (80.7, 89.3)
- moved U5 48.3 mm to (163.5, 94.9), turned to 90 degrees
- moved U3 43.8 mm to (109.9, 89.3)
- moved U2 34.2 mm to (66.1, 89.3)
- moved TP1 33.6 mm to (169.0, 80.6)
- moved R1 30.6 mm to (167.3, 84.0), turned to -90 degrees
- moved C11 23.5 mm to (133.5, 89.5), turned to 0 degrees
- moved C10 20.4 mm to (130.1, 89.5), turned to 180 degrees
- moved C9 13.0 mm to (118.9, 89.5), turned to 0 degrees
- moved C7 8.22 mm to (104.3, 89.5), turned to 0 degrees
- moved C5 7.32 mm to (89.7, 89.5), turned to 0 degrees
- moved C3 6.92 mm to (75.1, 89.5), turned to 0 degrees
- moved C1 6.53 mm to (60.5, 89.5), turned to 0 degrees
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Connections:
- J1 pad 18: /D16 -> /A0
- J1 pad 19: /D17 -> /A1
- J1 pad 20: /D18 -> /A2
- J1 pad 21: /D19 -> /A3
- J1 pad 22: /D20 -> /A4
- J1 pad 23: /D21 -> /A5
- J1 pad 24: /D22 -> /A6
- J1 pad 25: /D23 -> /A7
- J1 pad 26: /A0 -> /A8
- J1 pad 27: /A1 -> /A9
- J1 pad 28: /A2 -> /A10
- J1 pad 29: /A3 -> /A11
- J1 pad 30: /A4 -> /A12
- J1 pad 31: /A5 -> /D16
- J1 pad 32: /A6 -> /D17
- J1 pad 33: /A7 -> /D18
- J1 pad 34: /A8 -> /D19
- J1 pad 35: /A9 -> /D20
- J1 pad 36: /A10 -> /D21
- J1 pad 37: /A11 -> /D22
- J1 pad 38: /A12 -> /D23
- J1 pad 52: /~{SAS} -> /D24
- J1 pad 53: /~{SBS} -> /D25
- J1 pad 54: /PSCL -> /D26
- J1 pad 55: /PSDA -> /D27
- J1 pad 56: /D24 -> /D28
- J1 pad 57: /D25 -> /D29
- J1 pad 58: /D26 -> /D30
- J1 pad 59: /D27 -> /D31
- J1 pad 60: /D28 -> /D32
- J1 pad 61: /D29 -> /D33
- J1 pad 62: /D30 -> /D34
- J1 pad 63: /D31 -> /D35
- J1 pad 64: /D32 -> /D36
- J1 pad 65: /D33 -> /D37
- J1 pad 66: /D34 -> /D38
- J1 pad 67: /D35 -> /D39
- J1 pad 68: /D36 -> /D40
- J1 pad 69: /D37 -> /D41
- J1 pad 70: /D38 -> /D42
- J1 pad 71: /D39 -> /D43
- J1 pad 72: /D40 -> /D44
- J1 pad 73: /D41 -> /D45
- J1 pad 74: /D42 -> /D46
- J1 pad 75: /D43 -> /D47
- J1 pad 76: /D44 -> unconnected-(J1-NC-Pad76)
- J1 pad 77: /D45 -> unconnected-(J1-NC-Pad77)
- J1 pad 78: /D46 -> /PSCL
- J1 pad 79: /D47 -> /PSDA
- R1 pad 1: +5V -> Net-(U5-WP)
- R1 pad 2: Net-(U6-WP) -> +5V
- TP1 pad 1: Net-(U6-WP) -> Net-(U5-WP)
- U1 pad 1: /A0 -> /A18
- U1 pad 2: /A1 -> /A19
- U1 pad 3: /A2 -> unconnected-(U1-Y3-Pad3)
- U1 pad 4: /A3 -> GND
- U1 pad 5: /A4 -> /~{SCS}
- U1 pad 6: /~{SAS} -> /~{SBS}
- U1 pad 7: /D0 -> /~{SAS}
- U1 pad 8: /D1 -> +5V
- U2 pad 10: /D19 -> /D3
- U2 pad 13: /D20 -> /D4
- U2 pad 14: /D21 -> /D5
- U2 pad 15: /D22 -> /D6
- U2 pad 16: /D23 -> /D7
- U2 pad 29: /D24 -> /D8
- U2 pad 30: /D25 -> /D9
- U2 pad 31: /D26 -> /D10
- U2 pad 32: /D27 -> /D11
- U2 pad 35: /D28 -> /D12
- U2 pad 36: /D29 -> /D13
- U2 pad 37: /D30 -> /D14
- U2 pad 38: /D31 -> /D15
- U2 pad 7: /D16 -> /D0
- U2 pad 8: /D17 -> /D1
- U2 pad 9: /D18 -> /D2
- U3 pad 10: /D35 -> /D19
- U3 pad 13: /D36 -> /D20
- U3 pad 14: /D37 -> /D21
- U3 pad 15: /D38 -> /D22
- U3 pad 16: /D39 -> /D23
- U3 pad 29: /D40 -> /D24
- U3 pad 30: /D41 -> /D25
- U3 pad 31: /D42 -> /D26
- U3 pad 32: /D43 -> /D27
- U3 pad 35: /D44 -> /D28
- U3 pad 36: /D45 -> /D29
- U3 pad 37: /D46 -> /D30
- U3 pad 38: /D47 -> /D31
- U3 pad 7: /D32 -> /D16
- U3 pad 8: /D33 -> /D17
- U3 pad 9: /D34 -> /D18
- U4 pad 1: /A0 -> /A2
- U4 pad 10: /D3 -> /D35
- U4 pad 13: /D4 -> /D36
- U4 pad 14: /D5 -> /D37
- U4 pad 15: /D6 -> /D38
- U4 pad 16: /D7 -> /D39
- U4 pad 18: /A5 -> /A7
- U4 pad 19: /A6 -> /A8
- U4 pad 2: /A1 -> /A3
- U4 pad 20: /A7 -> /A9
- U4 pad 21: /A8 -> /A10
- U4 pad 22: /A9 -> /A11
- U4 pad 23: /A10 -> /A12
- U4 pad 24: /A11 -> /A13
- U4 pad 25: /A12 -> /A14
- U4 pad 26: /A13 -> /A15
- U4 pad 27: /A14 -> /A16
- U4 pad 29: /D8 -> /D40
- U4 pad 3: /A2 -> /A4
- U4 pad 30: /D9 -> /D41
- U4 pad 31: /D10 -> /D42
- U4 pad 32: /D11 -> /D43
- U4 pad 35: /D12 -> /D44
- U4 pad 36: /D13 -> /D45
- U4 pad 37: /D14 -> /D46
- U4 pad 38: /D15 -> /D47
- U4 pad 4: /A3 -> /A5
- U4 pad 42: /A15 -> /A17
- U4 pad 43: /A16 -> /A18
- U4 pad 44: /A17 -> /A19
- U4 pad 5: /A4 -> /A6
- U4 pad 6: /~{SBS} -> GND
- U4 pad 7: /D0 -> /D32
- U4 pad 8: /D1 -> /D33
- U4 pad 9: /D2 -> /D34
- U5 pad 1: /A0 -> GND
- U5 pad 2: /A1 -> GND
- U5 pad 3: /A2 -> GND
- U5 pad 4: /A3 -> GND
- U5 pad 5: /A4 -> /PSDA
- U5 pad 6: /~{SBS} -> /PSCL
- U5 pad 7: /D16 -> Net-(U5-WP)
- U5 pad 8: /D17 -> +5V
- U6 pad 1: GND -> /A0
- U6 pad 2: GND -> /A1
- U6 pad 3: GND -> /A2
- U6 pad 4: GND -> /A3
- U6 pad 5: /PSDA -> /A4
- U6 pad 6: /PSCL -> /~{SBS}
- U6 pad 7: Net-(U6-WP) -> /D0
- U6 pad 8: +5V -> /D1
Routing:
- net /~{SCS}: track 0.00 -> 86.7 mm, vias 0 -> 3
- net /A19: track 2.80 -> 61.4 mm
- net /A18: track 2.80 -> 60.5 mm
- net /A14: track 144.7 -> 101.7 mm, vias 7 -> 8
- net /~{SBS}: track 67.8 -> 95.3 mm, vias 4 -> 3
- net +5V: track 186.1 -> 162.6 mm, vias 16 -> 29
- net /PSCL: track 29.1 -> 8.56 mm, vias 3 -> 0
- net /PSDA: track 28.7 -> 8.56 mm, vias 3 -> 0
- net /D11: track 30.1 -> 48.3 mm, vias 3 -> 4
- net /D10: track 30.3 -> 47.1 mm, vias 3 -> 4
- net /D19: track 39.6 -> 56.1 mm
- net /A0: track 115.0 -> 98.6 mm
- net /D18: track 40.7 -> 56.5 mm
- net /D9: track 30.3 -> 46.0 mm, vias 3 -> 4
- net Net-(U5-WP): track 0.00 -> 15.4 mm
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Other:
- board text added: "--- WP DIS - - WP ENA"
