File: kicad/projects/m68k-hbc/IO.kicad_sch (KiCad schematic)
At the start: 25 parts, among them J11 KMDGX-6SG_P-S4N, J6 5747840-4, U13 MAX232, U14 68681, U17 VT82C42, U35 74LS06, U41 68230, X5 8M, Y1 3.6864M, Y2 8M

Commit message: Modified system architecture, New KiCad Project: Cache Memory Module(SIMM80)
Parts:
- removed C14: 100p, Capacitor_SMD:C_1206_3216Metric_Pad1.33x1.80mm_HandSolder, symbol Device:C
- removed C4, C5: 10p, Capacitor_SMD:C_1206_3216Metric_Pad1.33x1.80mm_HandSolder, symbol Device:C
- removed U14: 68681, Package_DIP:DIP-40_W15.24mm_Socket, symbol Interface:68681
- removed U41: 68230, Package_DIP:DIP-48_W15.24mm_Socket, symbol Interface:68230
- removed X5: 8M, Oscillator:Oscillator_SMD_SeikoEpson_SG8002CA-4Pin_7.0x5.0mm, symbol Oscillator:SG-8002CA
- removed Y1: 3.6864M, Crystal:Crystal_HC52-6mm_Vertical, symbol Device:Crystal
- added IC3: MC68901P, Package_DIP:DIP-48_W15.24mm_Socket, symbol micro-mc68000:MC68901P
- C14: value 100p -> 100n
Connections:
- net +5V: now also C14.1, IC3.11 (VCC); no longer C14.2
- net A0: now also IC3.2 (RS1)
- net A1: now also IC3.3 (RS2)
- net A2: now also IC3.4 (RS3)
- net A3: now also IC3.5 (RS4)
- net A4: now also IC3.6 (RS5)
- net D24: now also IC3.37 (D0)
- net D25: now also IC3.38 (D1)
- net D26: now also IC3.39 (D2)
- net D27: now also IC3.40 (D3)
- net D28: now also IC3.41 (D4)
- net D29: now also IC3.42 (D5)
- net D30: now also IC3.43 (D6)
- net D31: now also IC3.44 (D7)
- net GND: now also C14.2, IC3.36 (GND); no longer C14.1
- net R/~{W}: now also IC3.1 (R/W\)
- net ~{DTACK8}: now also IC3.46 (DTACK)
- net ~{IACK}: now also IC3.45 (IACK)
- net ~{PERRST}: now also IC3.21 (RESET)
- net ~{TIMCS}: now also IC3.48 (CS)
- net at U13.11 (T1IN): now also IC3.8 (SO)
- net at U13.12 (R1OUT): now also IC3.9 (SI)
- new net CLK_4M: IC3.35 (CLK)
- new net TIMCLK: IC3.17 (XTAL1)
- new net ~{DS}: IC3.47 (DS)
- new net ~{MFPIRQ}: IC3.32 (IRQ)
- no-connect marks 10 -> 14
Other:
- moved on the sheet: C14

Commit message: Some Updates
Parts:
- C? (x3): renamed from C14; value 100n -> C; footprint Capacitor_SMD:C_1206_3216Metric_Pad1.33x1.80mm_HandSolder -> Capacitor_SMD:C_0603_1608Metric_Pad1.08x0.95mm_HandSolder
- C?: renamed from C6; value 1u -> C; footprint Capacitor_SMD:C_1206_3216Metric_Pad1.33x1.80mm_HandSolder -> Capacitor_SMD:C_0603_1608Metric_Pad1.08x0.95mm_HandSolder
- C?: renamed from C8; value 20p -> C; footprint Capacitor_SMD:C_1206_3216Metric_Pad1.33x1.80mm_HandSolder -> Capacitor_SMD:C_0603_1608Metric_Pad1.08x0.95mm_HandSolder
- C?: renamed from C2; value 1u -> C; footprint Capacitor_SMD:C_1206_3216Metric_Pad1.33x1.80mm_HandSolder -> Capacitor_SMD:C_0603_1608Metric_Pad1.08x0.95mm_HandSolder
- C?: renamed from C1; value 1u -> C; footprint Capacitor_SMD:C_1206_3216Metric_Pad1.33x1.80mm_HandSolder -> Capacitor_SMD:C_0603_1608Metric_Pad1.08x0.95mm_HandSolder
- C?: renamed from C3; value 1u -> C; footprint Capacitor_SMD:C_1206_3216Metric_Pad1.33x1.80mm_HandSolder -> Capacitor_SMD:C_0603_1608Metric_Pad1.08x0.95mm_HandSolder
- C?: renamed from C9; value 20p -> C; footprint Capacitor_SMD:C_1206_3216Metric_Pad1.33x1.80mm_HandSolder -> Capacitor_SMD:C_0603_1608Metric_Pad1.08x0.95mm_HandSolder
- C?: renamed from C7; value 1u -> C; footprint Capacitor_SMD:C_1206_3216Metric_Pad1.33x1.80mm_HandSolder -> Capacitor_SMD:C_0603_1608Metric_Pad1.08x0.95mm_HandSolder
- IC4: renamed from IC3; footprint Package_DIP:DIP-48_W15.24mm_Socket -> Package_DIP:DIP-48_W15.24mm
- J?: renamed from J11; footprint KMDGX6SGPS4N:KMDGX6SGPS4N -> KMDGX6SGPS4N
- J?: renamed from J6; footprint 57478404:57478404 -> 57478404
- R?: renamed from R2; value 10k -> R; footprint Resistor_SMD:R_1206_3216Metric_Pad1.30x1.75mm_HandSolder -> Resistor_SMD:R_0603_1608Metric_Pad0.98x0.95mm_HandSolder
- R?: renamed from R1; value 10k -> R; footprint Resistor_SMD:R_1206_3216Metric_Pad1.30x1.75mm_HandSolder -> Resistor_SMD:R_0603_1608Metric_Pad0.98x0.95mm_HandSolder
- U?: renamed from U17; footprint Package_DIP:DIP-40_W15.24mm -> Package_DIP:DIP-40_W15.24mm_Socket
- Y?: renamed from Y2; value 8M -> Crystal
- renumbered U35 to U?, U13 to U?
Connections:
- net A0 renamed OPB_A0
- net A1 renamed OPB_A1
- net A2 renamed OPB_A2
- net A3 renamed OPB_A3
- net A4 renamed OPB_A4
- net D24 renamed OPB_D0
- net D25 renamed OPB_D1
- net D26 renamed OPB_D2
- net D27 renamed OPB_D3
- net D28 renamed OPB_D4
- net D29 renamed OPB_D5
- net D30 renamed OPB_D6
- net D31 renamed OPB_D7
- net R/~{W} renamed OPB_R/~{W}
- net ~{8242CS} renamed ~{CS_8242}
- net ~{DS} renamed ~{OPB_DS}
- net ~{DTACK8} renamed ~{OPB_DTACK8}
- net ~{IACK} renamed ~{IACK_68901}
- net ~{KBIRQ} renamed ~{IRQ_KB}
- net ~{MFPIRQ} renamed ~{IRQ_68901}
- net ~{MSIRQ} renamed ~{IRQ_MS}
- net ~{PERRST} renamed ~{RST_68901}
- net ~{RST_68901}: no longer U?.4 (~{RST})
- net ~{RD} renamed ~{OPB_RD}
- net ~{TIMCS} renamed ~{CS_68901}
- net ~{WR} renamed ~{OPB_WR}
- new net ~{RST_8242}: U?.4 (~{RST})
Other:
- note added: "OPB Signals"
- moved on the sheet: C?, IC4A, IC4B, J?, R?, U?, U?A, U?B, U?C, U?D, U?E, U?F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
