File: kicad/projects/m68k-hbc/Audio.kicad_sch (KiCad schematic)
At the start: 0 parts

Commit message: Modified system architecture, New KiCad Project: Cache Memory Module(SIMM80)
Parts:
- added C100, C102, C106, C95: 33p, Capacitor_SMD:C_1206_3216Metric_Pad1.33x1.80mm_HandSolder, symbol Device:C
- added C101, C109, C113, C87, C89: 10u, Capacitor_THT:CP_Radial_D5.0mm_P2.50mm, symbol Device:C_Polarized
- added C103, C108, C115, C78: 47p, Capacitor_SMD:C_1206_3216Metric_Pad1.33x1.80mm_HandSolder, symbol Device:C
- added C104, C77: 1.2n, Capacitor_SMD:C_1206_3216Metric_Pad1.33x1.80mm_HandSolder, symbol Device:C
- added C105, C107, C79, C80, C83, C84, C85, C88: 100n, Capacitor_SMD:C_1206_3216Metric_Pad1.33x1.80mm_HandSolder, symbol Device:C
- added C110, C114: 1.8n, Capacitor_SMD:C_1206_3216Metric_Pad1.33x1.80mm_HandSolder, symbol Device:C
- added C111, C112, C90, C91, C98, C99: 1u, Capacitor_SMD:C_1206_3216Metric_Pad1.33x1.80mm_HandSolder, symbol Device:C
- added C116: 100n, Capacitor_SMD:C_1210_3225Metric, symbol Device:C
- added C81, C82, C86: 1u, Capacitor_THT:CP_Radial_D5.0mm_P2.50mm, symbol Device:C_Polarized
- added C92, C93, C96, C97: 1u, Capacitor_THT:CP_Radial_D5.0mm_P2.50mm, symbol Device:C_Feedthrough
- added C94: 470n, Capacitor_SMD:C_1206_3216Metric_Pad1.33x1.80mm_HandSolder, symbol Device:C
- added FB3: FerriteBead, Inductor_THT:L_Axial_L5.3mm_D2.2mm_P2.54mm_Vertical_Vishay_IM-1, symbol Device:FerriteBead
- added J19: STX-4335-5BGP-S1, STX43355BGPS1:STX43355BGPS1, symbol STX-4335-5BGP-S1:STX-4335-5BGP-S1
- added L2, L3, L4, L5, L6, L7: L, Inductor_SMD:L_1206_3216Metric_Pad1.42x1.75mm_HandSolder, symbol Device:L
- added R12: 2, Resistor_SMD:R_1206_3216Metric_Pad1.30x1.75mm_HandSolder, symbol Device:R
- added R13, R22: 1.5k, Resistor_SMD:R_1206_3216Metric_Pad1.30x1.75mm_HandSolder, symbol Device:R
- added R14, R24: 11k, Resistor_SMD:R_1206_3216Metric_Pad1.30x1.75mm_HandSolder, symbol Device:R
- added R15, R23: 22k, Resistor_SMD:R_1206_3216Metric_Pad1.30x1.75mm_HandSolder, symbol Device:R
- added R16, R17, R19, R21: 47k, Resistor_SMD:R_1206_3216Metric_Pad1.30x1.75mm_HandSolder, symbol Device:R
- added R18, R20: 5.1k, Resistor_SMD:R_1206_3216Metric_Pad1.30x1.75mm_HandSolder, symbol Device:R
- added R25, R32: 18k, Resistor_SMD:R_1206_3216Metric_Pad1.30x1.75mm_HandSolder, symbol Device:R
- added R26, R30: 680, Resistor_SMD:R_1206_3216Metric_Pad1.30x1.75mm_HandSolder, symbol Device:R
- added R27, R31: 8.2k, Resistor_SMD:R_1206_3216Metric_Pad1.30x1.75mm_HandSolder, symbol Device:R
- added R28, R29: 75, Resistor_SMD:R_1206_3216Metric_Pad1.30x1.75mm_HandSolder, symbol Device:R
- added U18, U19: MC33078, Package_DIP:DIP-8_W7.62mm_Socket, symbol Amplifier_Operational:MC33078
- added U20: CS4231A, Package_LCC:PLCC-68_THT-Socket, symbol m68k-hbc-ic:CS4231A
- added U21: NE5532, Package_DIP:DIP-8_W7.62mm_Socket, symbol Amplifier_Operational:NE5532
- added Y5: 24.576M, Crystal:Crystal_HC52-6mm_Vertical, symbol Device:Crystal
- added Y6: 16.9344M, Crystal:Crystal_HC52-6mm_Vertical, symbol Device:Crystal
Connections:
- new net: C108.2, R25.2, R28.1, U21.1
- new net: C108.1, R25.1, R27.2, U21.2 (-)
- new net: C96.2, R19.2, U18.5 (+)
- new net: C115.1, R31.2, R32.1, U21.6 (-)
- new net: C115.2, R29.1, R32.2, U21.7
- new net: C93.1, C93.3, L3.2
- new net: C109.1, C110.1, R26.2
- new net: C109.2, R27.1
- new net: C106.1, U20.22 (XTAL2O), Y6.1
- new net: C102.1, U20.21 (XTAL2I), Y6.2
- new net: C92.1, C92.3, L2.2
- new net: C101.1, R22.1
- new net: C113.1, C114.1, R30.2
- new net: C113.2, R31.1
- new net: C95.1, U20.17 (XTAL1I), Y5.2
- new net: L6.1, R28.2
- new net: C77.2, C90.1, R14.2, U18.1
- new net: C97.1, C97.3, L5.2
- new net: C97.2, R21.1
- new net: L7.1, R29.2
- new net: C104.1, R22.2, R24.1, U18.6 (-)
- new net: C104.2, C98.1, R24.2, U18.7
- new net: R20.2, R21.2, U19.5 (+)
- new net: C100.1, U20.18 (XTAL1O), Y5.1
- new net: C93.2, R16.1
- new net: C77.1, R13.2, R14.1, U18.2 (-)
- new net: C78.1, R15.1, U19.2 (-)
- new net: C78.2, C91.1, R15.2, U19.1
- new net: R16.2, R18.1, U19.3 (+)
- new net: U20.24 (NC), U20.25 (NC), U20.44 (NC), U20.45 (NC), U20.48 (NC), U20.54 (NC)
- new net: C112.1, U20.26 (RFILT)
- new net: C111.1, U20.31 (LFILT)
- new net: C94.2, U20.32 (VREF)
- new net: C88.1, C89.1, U20.33 (VREFI)
- new net: C92.2, R17.1, U18.3 (+)
- new net: C87.1, R13.1
- new net: C103.1, R23.1, U19.6 (-)
- new net: C103.2, C99.1, R23.2, U19.7
- new net: C96.1, C96.3, L4.2
- new net +12V: C116.1, U21.8 (V+)
- new net +5V: C79.1, C80.1, C81.1, C82.1, FB3.1, U20.1 (VD1), U20.7 (VD2)
- new net +5VA: C105.1, C107.1, C85.1, C86.1, R12.2, U18.8 (V+), U19.8 (V+), U20.35 (VA1), U20.36 (VA2)
- new net -12V: C116.2, U21.4 (V-)
- new net A0: U20.10 (A0)
- new net A1: U20.9 (A1)
- new net AUDIOIRQ: U20.57 (IRQ)
- new net BLUERING: J19.35, L3.1
- new net BLUETIP: J19.32, L5.1
- new net D24: U20.6 (D0)
- new net D25: U20.5 (D1)
- new net D26: U20.4 (D2)
- new net D27: U20.3 (D3)
- new net D28: U20.68 (D4)
- new net D29: U20.67 (D5)
- new net D30: U20.66 (D6)
- new net D31: U20.65 (D7)
- new net GND: C100.2, C102.2, C106.2, C79.2, C80.2, C81.2, C82.2, C94.1, C95.2, R17.2, R18.2, R19.1, R20.1, U20.2 (DGND1), U20.55 (TEST), U20.8 (DGND2)
- new net GNDA: C101.2, C105.2, C107.2, C110.2, C111.2, C112.2, C114.2, C83.2, C84.2, C85.2, C86.2, C87.2, C88.2, C89.2, J19.1, J19.3, J19.33, J19.34, J19.4, U18.4 (V-), U19.4 (V-), U20.16 (DGND3), U20.20 (DGND4), U20.34 (AGND1), U20.37 (AGND2), U20.53 (DGND7), U20.64 (DGND8), U21.3 (+), U21.5 (+)
- new net GNDPWR: J19.MH1, J19.MH2, J19.MH3, J19.MH4
- new net LAUX1: U20.39 (LAUX1)
- new net LAUX2: U20.38 (LAUX2)
- new net LIMERING: J19.25, L6.2
- new net LIMETIP: J19.22, L7.2
- new net LLINE: C99.2, U20.30 (LLINE)
- new net LMIC: C90.2, U20.29 (LMIC)
- new net LOUT: R30.1, U20.40 (LOUT)
- new net MIN: U20.46 (MIN)
- new net MOUT: U20.47 (MOUT)
- new net PINKRING: J19.5, L4.1
- new net PINKTIP: J19.2, L2.1
- new net RAUX1: U20.42 (RAUX1)
- new net RAUX2: U20.43 (RAUX2)
- new net RLINE: C91.2, U20.27 (RLINE)
- new net RMIC: C98.2, U20.28 (RMIC)
- new net ROUT: R26.1, U20.41 (ROUT)
- new net VD34: C83.1, C84.1, FB3.2, R12.1, U20.15 (VD3), U20.19 (VD4), U20.23 (~{PDWN})
- new net ~{AUDIOCS}: U20.59 (~{CS})
- new net ~{RD}: U20.60 (~{RD})
- new net ~{WR}: U20.61 (~{WR})
Other:
- note added: "TODO: Assert ~{DTACK8} after 60ns of ~{RD} assertion"

Commit message: Some Updates
Parts:
- C100: renamed from C94; value 470n -> C; footprint Capacitor_SMD:C_1206_3216Metric_Pad1.33x1.80mm_HandSolder -> Capacitor_SMD:C_0603_1608Metric_Pad1.08x0.95mm_HandSolder
- C101: renamed from C95; value 33p -> C; footprint Capacitor_SMD:C_1206_3216Metric_Pad1.33x1.80mm_HandSolder -> Capacitor_SMD:C_0603_1608Metric_Pad1.08x0.95mm_HandSolder
- C102: renamed from C96; value 1u -> C_Feedthrough
- C103: renamed from C97; value 1u -> C_Feedthrough
- C104: renamed from C98; value 1u -> C; footprint Capacitor_SMD:C_1206_3216Metric_Pad1.33x1.80mm_HandSolder -> Capacitor_SMD:C_0603_1608Metric_Pad1.08x0.95mm_HandSolder
- C105: renamed from C99; value 1u -> C; footprint Capacitor_SMD:C_1206_3216Metric_Pad1.33x1.80mm_HandSolder -> Capacitor_SMD:C_0603_1608Metric_Pad1.08x0.95mm_HandSolder
- C106: renamed from C100; value 33p -> C; footprint Capacitor_SMD:C_1206_3216Metric_Pad1.33x1.80mm_HandSolder -> Capacitor_SMD:C_0603_1608Metric_Pad1.08x0.95mm_HandSolder
- C107: renamed from C101; value 10u -> C_Polarized
- C108: renamed from C102; value 33p -> C; footprint Capacitor_SMD:C_1206_3216Metric_Pad1.33x1.80mm_HandSolder -> Capacitor_SMD:C_0603_1608Metric_Pad1.08x0.95mm_HandSolder
- C109: renamed from C103; value 47p -> C; footprint Capacitor_SMD:C_1206_3216Metric_Pad1.33x1.80mm_HandSolder -> Capacitor_SMD:C_0603_1608Metric_Pad1.08x0.95mm_HandSolder
- C110: renamed from C104; value 1.2n -> C; footprint Capacitor_SMD:C_1206_3216Metric_Pad1.33x1.80mm_HandSolder -> Capacitor_SMD:C_0603_1608Metric_Pad1.08x0.95mm_HandSolder
- C111: renamed from C105; value 100n -> C; footprint Capacitor_SMD:C_1206_3216Metric_Pad1.33x1.80mm_HandSolder -> Capacitor_SMD:C_0603_1608Metric_Pad1.08x0.95mm_HandSolder
- C112: renamed from C106; value 33p -> C; footprint Capacitor_SMD:C_1206_3216Metric_Pad1.33x1.80mm_HandSolder -> Capacitor_SMD:C_0603_1608Metric_Pad1.08x0.95mm_HandSolder
- C113: renamed from C107; value 100n -> C; footprint Capacitor_SMD:C_1206_3216Metric_Pad1.33x1.80mm_HandSolder -> Capacitor_SMD:C_0603_1608Metric_Pad1.08x0.95mm_HandSolder
- C114: renamed from C108; value 47p -> C; footprint Capacitor_SMD:C_1206_3216Metric_Pad1.33x1.80mm_HandSolder -> Capacitor_SMD:C_0603_1608Metric_Pad1.08x0.95mm_HandSolder
- C115: renamed from C109; value 10u -> C_Polarized
- C116: renamed from C110; value 1.8n -> C; footprint Capacitor_SMD:C_1206_3216Metric_Pad1.33x1.80mm_HandSolder -> Capacitor_SMD:C_0603_1608Metric_Pad1.08x0.95mm_HandSolder
- C117: renamed from C111; value 1u -> C; footprint Capacitor_SMD:C_1206_3216Metric_Pad1.33x1.80mm_HandSolder -> Capacitor_SMD:C_0603_1608Metric_Pad1.08x0.95mm_HandSolder
- C118: renamed from C112; value 1u -> C; footprint Capacitor_SMD:C_1206_3216Metric_Pad1.33x1.80mm_HandSolder -> Capacitor_SMD:C_0603_1608Metric_Pad1.08x0.95mm_HandSolder
- C119: renamed from C113; value 10u -> C_Polarized
- C120: renamed from C114; value 1.8n -> C; footprint Capacitor_SMD:C_1206_3216Metric_Pad1.33x1.80mm_HandSolder -> Capacitor_SMD:C_0603_1608Metric_Pad1.08x0.95mm_HandSolder
- C121: renamed from C115; value 47p -> C; footprint Capacitor_SMD:C_1206_3216Metric_Pad1.33x1.80mm_HandSolder -> Capacitor_SMD:C_0603_1608Metric_Pad1.08x0.95mm_HandSolder
- C122: renamed from C116; value 100n -> C; footprint Capacitor_SMD:C_1210_3225Metric -> Capacitor_SMD:C_0603_1608Metric_Pad1.08x0.95mm_HandSolder
- C83: renamed from C77; value 1.2n -> C; footprint Capacitor_SMD:C_1206_3216Metric_Pad1.33x1.80mm_HandSolder -> Capacitor_SMD:C_0603_1608Metric_Pad1.08x0.95mm_HandSolder
- C84: renamed from C78; value 47p -> C; footprint Capacitor_SMD:C_1206_3216Metric_Pad1.33x1.80mm_HandSolder -> Capacitor_SMD:C_0603_1608Metric_Pad1.08x0.95mm_HandSolder
- C85: renamed from C79; value 100n -> C; footprint Capacitor_SMD:C_1206_3216Metric_Pad1.33x1.80mm_HandSolder -> Capacitor_SMD:C_0603_1608Metric_Pad1.08x0.95mm_HandSolder
- C86: renamed from C80; value 100n -> C; footprint Capacitor_SMD:C_1206_3216Metric_Pad1.33x1.80mm_HandSolder -> Capacitor_SMD:C_0603_1608Metric_Pad1.08x0.95mm_HandSolder
- C87: renamed from C81; value 1u -> C_Polarized
- C88: renamed from C82; value 1u -> C_Polarized
- C89: renamed from C83; value 100n -> C; footprint Capacitor_SMD:C_1206_3216Metric_Pad1.33x1.80mm_HandSolder -> Capacitor_SMD:C_0603_1608Metric_Pad1.08x0.95mm_HandSolder
- C90: renamed from C84; value 100n -> C; footprint Capacitor_SMD:C_1206_3216Metric_Pad1.33x1.80mm_HandSolder -> Capacitor_SMD:C_0603_1608Metric_Pad1.08x0.95mm_HandSolder
- C91: renamed from C85; value 100n -> C; footprint Capacitor_SMD:C_1206_3216Metric_Pad1.33x1.80mm_HandSolder -> Capacitor_SMD:C_0603_1608Metric_Pad1.08x0.95mm_HandSolder
- C92: renamed from C86; value 1u -> C_Polarized
- C93: renamed from C87; value 10u -> C_Polarized
- C94: renamed from C88; value 100n -> C; footprint Capacitor_SMD:C_1206_3216Metric_Pad1.33x1.80mm_HandSolder -> Capacitor_SMD:C_0603_1608Metric_Pad1.08x0.95mm_HandSolder
- C95: renamed from C89; value 10u -> C_Polarized
- C96: renamed from C90; value 1u -> C; footprint Capacitor_SMD:C_1206_3216Metric_Pad1.33x1.80mm_HandSolder -> Capacitor_SMD:C_0603_1608Metric_Pad1.08x0.95mm_HandSolder
- C97: renamed from C91; value 1u -> C; footprint Capacitor_SMD:C_1206_3216Metric_Pad1.33x1.80mm_HandSolder -> Capacitor_SMD:C_0603_1608Metric_Pad1.08x0.95mm_HandSolder
- C98: renamed from C92; value 1u -> C_Feedthrough
- C99: renamed from C93; value 1u -> C_Feedthrough
- J17: renamed from J19; footprint STX43355BGPS1:STX43355BGPS1 -> STX43355BGPS1
- R10: renamed from R12; value 2 -> R; footprint Resistor_SMD:R_1206_3216Metric_Pad1.30x1.75mm_HandSolder -> Resistor_SMD:R_0603_1608Metric_Pad0.98x0.95mm_HandSolder
- R11: renamed from R13; value 1.5k -> R; footprint Resistor_SMD:R_1206_3216Metric_Pad1.30x1.75mm_HandSolder -> Resistor_SMD:R_0603_1608Metric_Pad0.98x0.95mm_HandSolder
- R12: renamed from R14; value 11k -> R; footprint Resistor_SMD:R_1206_3216Metric_Pad1.30x1.75mm_HandSolder -> Resistor_SMD:R_0603_1608Metric_Pad0.98x0.95mm_HandSolder
- R13: renamed from R15; value 22k -> R; footprint Resistor_SMD:R_1206_3216Metric_Pad1.30x1.75mm_HandSolder -> Resistor_SMD:R_0603_1608Metric_Pad0.98x0.95mm_HandSolder
- R14: renamed from R16; value 47k -> R; footprint Resistor_SMD:R_1206_3216Metric_Pad1.30x1.75mm_HandSolder -> Resistor_SMD:R_0603_1608Metric_Pad0.98x0.95mm_HandSolder
- R15: renamed from R17; value 47k -> R; footprint Resistor_SMD:R_1206_3216Metric_Pad1.30x1.75mm_HandSolder -> Resistor_SMD:R_0603_1608Metric_Pad0.98x0.95mm_HandSolder
- R16: renamed from R18; value 5.1k -> R; footprint Resistor_SMD:R_1206_3216Metric_Pad1.30x1.75mm_HandSolder -> Resistor_SMD:R_0603_1608Metric_Pad0.98x0.95mm_HandSolder
- R17: renamed from R19; value 47k -> R; footprint Resistor_SMD:R_1206_3216Metric_Pad1.30x1.75mm_HandSolder -> Resistor_SMD:R_0603_1608Metric_Pad0.98x0.95mm_HandSolder
- R18: renamed from R20; value 5.1k -> R; footprint Resistor_SMD:R_1206_3216Metric_Pad1.30x1.75mm_HandSolder -> Resistor_SMD:R_0603_1608Metric_Pad0.98x0.95mm_HandSolder
- R19: renamed from R21; value 47k -> R; footprint Resistor_SMD:R_1206_3216Metric_Pad1.30x1.75mm_HandSolder -> Resistor_SMD:R_0603_1608Metric_Pad0.98x0.95mm_HandSolder
- R20: renamed from R22; value 1.5k -> R; footprint Resistor_SMD:R_1206_3216Metric_Pad1.30x1.75mm_HandSolder -> Resistor_SMD:R_0603_1608Metric_Pad0.98x0.95mm_HandSolder
- R21: renamed from R23; value 22k -> R; footprint Resistor_SMD:R_1206_3216Metric_Pad1.30x1.75mm_HandSolder -> Resistor_SMD:R_0603_1608Metric_Pad0.98x0.95mm_HandSolder
- R22: renamed from R24; value 11k -> R; footprint Resistor_SMD:R_1206_3216Metric_Pad1.30x1.75mm_HandSolder -> Resistor_SMD:R_0603_1608Metric_Pad0.98x0.95mm_HandSolder
- R23: renamed from R25; value 18k -> R; footprint Resistor_SMD:R_1206_3216Metric_Pad1.30x1.75mm_HandSolder -> Resistor_SMD:R_0603_1608Metric_Pad0.98x0.95mm_HandSolder
- R24: renamed from R26; value 680 -> R; footprint Resistor_SMD:R_1206_3216Metric_Pad1.30x1.75mm_HandSolder -> Resistor_SMD:R_0603_1608Metric_Pad0.98x0.95mm_HandSolder
- R25: renamed from R27; value 8.2k -> R; footprint Resistor_SMD:R_1206_3216Metric_Pad1.30x1.75mm_HandSolder -> Resistor_SMD:R_0603_1608Metric_Pad0.98x0.95mm_HandSolder
- R26: renamed from R28; value 75 -> R; footprint Resistor_SMD:R_1206_3216Metric_Pad1.30x1.75mm_HandSolder -> Resistor_SMD:R_0603_1608Metric_Pad0.98x0.95mm_HandSolder
- R27: renamed from R29; value 75 -> R; footprint Resistor_SMD:R_1206_3216Metric_Pad1.30x1.75mm_HandSolder -> Resistor_SMD:R_0603_1608Metric_Pad0.98x0.95mm_HandSolder
- R28: renamed from R30; value 680 -> R; footprint Resistor_SMD:R_1206_3216Metric_Pad1.30x1.75mm_HandSolder -> Resistor_SMD:R_0603_1608Metric_Pad0.98x0.95mm_HandSolder
- R29: renamed from R31; value 8.2k -> R; footprint Resistor_SMD:R_1206_3216Metric_Pad1.30x1.75mm_HandSolder -> Resistor_SMD:R_0603_1608Metric_Pad0.98x0.95mm_HandSolder
- R30: renamed from R32; value 18k -> R; footprint Resistor_SMD:R_1206_3216Metric_Pad1.30x1.75mm_HandSolder -> Resistor_SMD:R_0603_1608Metric_Pad0.98x0.95mm_HandSolder
- U24: renamed from U20; footprint Package_LCC:PLCC-68_THT-Socket -> Package_LCC:PLCC-68
- Y5: value 24.576M -> Crystal
- Y6: value 16.9344M -> Crystal
- renumbered FB3 to FB1, L2 to L1, L3 to L2, L4 to L3, L5 to L4, L6 to L5, L7 to L6, U18 to U22, U19 to U23, U21 to U25
Connections:
- net GNDA: now also J17.23, J17.24
- net DACK_ACC: now reaches U24.11 (~{CDAK})
- net DRQ_ACC: now reaches U24.12 (CDRQ)
- net DACK_ACP: now reaches U24.13 (~{PDAK})
- net DRQ_ACP: now reaches U24.14 (PDRQ)
- net A0 renamed OPB_A0
- net A1 renamed OPB_A1
- net AUDIOIRQ renamed IRQ_ACODEC
- net D24 renamed OPB_D0
- net D25 renamed OPB_D1
- net D26 renamed OPB_D2
- net D27 renamed OPB_D3
- net D28 renamed OPB_D4
- net D29 renamed OPB_D5
- net D30 renamed OPB_D6
- net D31 renamed OPB_D7
- net ~{AUDIOCS} renamed ~{CS_ACODEC}
- net ~{RD} renamed ~{OPB_RD}
- net ~{WR} renamed ~{OPB_WR}
Other:
- note added: "OPB Signals"
- moved on the sheet: C102, C103, C104, C105, C107, C109, C110, C111, C113, C114, C115, C116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

Commit message: Large changes: EHBCSimpleEmu, kicad, fwcode, docs
This commit contains some large changes:
- Removed EHBCSimpleEmu (Moved to kms1212/llemu, kms1212/qemu)
- (likely) Removed fwcode; now it only boots and stops
- Modified documents
Parts:
- removed C100, C101, C104, C105, C106, C108, C109, C110, C111, C112, C113, C114, C116, C117, C118, C120, C121, C122, C83, C84, C85, C86, C89, C90, C91, C94, C96, C97: C, Capacitor_SMD:C_0603_1608Metric_Pad1.08x0.95mm_HandSolder, symbol Device:C
- removed C102, C103, C98, C99: C_Feedthrough, Capacitor_THT:CP_Radial_D5.0mm_P2.50mm, symbol Device:C_Feedthrough
- removed C107, C115, C119, C87, C88, C92, C93, C95: C_Polarized, Capacitor_THT:CP_Radial_D5.0mm_P2.50mm, symbol Device:C_Polarized
- removed FB1: FerriteBead, Inductor_THT:L_Axial_L5.3mm_D2.2mm_P2.54mm_Vertical_Vishay_IM-1, symbol Device:FerriteBead
- removed J17: STX-4335-5BGP-S1, STX43355BGPS1, symbol STX-4335-5BGP-S1:STX-4335-5BGP-S1
- removed L1, L2, L3, L4, L5, L6: L, Inductor_SMD:L_1206_3216Metric_Pad1.42x1.75mm_HandSolder, symbol Device:L
- removed R10, R11, R12, R13, R14, R15, R16, R17, R18, R19, R20, R21, R22, R23, R24, R25, R26, R27, R28, R29, R30: R, Resistor_SMD:R_0603_1608Metric_Pad0.98x0.95mm_HandSolder, symbol Device:R
- removed U22, U23: MC33078, Package_DIP:DIP-8_W7.62mm_Socket, symbol Amplifier_Operational:MC33078
- removed U24: CS4231A, Package_LCC:PLCC-68, symbol m68k-hbc-ic:CS4231A
- removed U25: NE5532, Package_DIP:DIP-8_W7.62mm_Socket, symbol Amplifier_Operational:NE5532
- removed Y5, Y6: Crystal, Crystal:Crystal_HC52-6mm_Vertical, symbol Device:Crystal
- added J9: STX-4335-5BGP-S1, STX43355BGPS1:STX43355BGPS1, symbol STX-4335-5BGP-S1:STX-4335-5BGP-S1
- added U12: CS4231A, Package_LCC:PLCC-68_THT-Socket, symbol m68k-hbc-ic:CS4231A
Connections:
- new net: U12.24 (NC), U12.25 (NC), U12.44 (NC), U12.45 (NC), U12.48 (NC), U12.54 (NC)
- new net A0: U12.10 (A0)
- new net A1: U12.9 (A1)
- new net D0: U12.6 (D0)
- new net D1: U12.5 (D1)
- new net D2: U12.4 (D2)
- new net D3: U12.3 (D3)
- new net D4: U12.68 (D4)
- new net D5: U12.67 (D5)
- new net D6: U12.66 (D6)
- new net D7: U12.65 (D7)
- new net ~{CS}: U12.59 (~{CS})
- new net ~{RD}: U12.60 (~{RD})
- new net ~{WR}: U12.61 (~{WR})
Other:
- note removed: "OPB Signals"
- note removed: "TODO: Assert ~{DTACK8} after 60ns of ~{RD} assertion"
