File: kicad/projects/m68k-hbc/CDC.kicad_sch (KiCad schematic)
At the start: 24 parts, among them J1 SIMM80_Cache, U1 CDC, U21 SIMM72, U22 SIMM72, U23 SIMM72, U24 SIMM72

Commit message: Large changes: EHBCSimpleEmu, kicad, fwcode, docs
This commit contains some large changes:
- Removed EHBCSimpleEmu (Moved to kms1212/llemu, kms1212/qemu)
- (likely) Removed fwcode; now it only boots and stops
- Modified documents
Parts:
- removed C18, C19, C20, C21, C22, C23, C24, C25, C26, C27, C28, C29, C30, C31, C32, C33, C34, C35: C, Capacitor_SMD:C_0603_1608Metric_Pad1.08x0.95mm_HandSolder, symbol Device:C
- removed J1: SIMM80_Cache, 5822030-4:58220304, symbol m68k-hbc-conn:SIMM80_Cache
- removed U1: CDC, Package_QFP:PQFP-240_32.1x32.1mm_P0.5mm, symbol m68k-hbc-ic:EPF6016QC240
- removed U21, U22, U23, U24: SIMM72, Sockets:SIM72, symbol m68k-hbc-ic:SIMM72
- added U18: EPF6016QC240, Package_QFP:PQFP-240_32.1x32.1mm_P0.5mm, symbol m68k-hbc-ic:EPF6016QC240
Connections:
- net A0: now also U18.197 (IO)
- net A1: now also U18.203 (IO)
- net A10: now also U18.224 (IO)
- net A11: now also U18.231 (IO)
- net A12: now also U18.226 (IO)
- net A13: now also U18.223 (IO)
- net A14: now also U18.225 (IO)
- net A15: now also U18.222 (IO)
- net A16: now also U18.220 (IO)
- net A17: now also U18.221 (IO)
- net A18: now also U18.218 (IO)
- net A19: now also U18.219 (IO)
- net A2: now also U18.237 (IO)
- net A20: now also U18.217 (IO)
- net A21: now also U18.215 (IO)
- net A22: now also U18.214 (IO)
- net A23: now also U18.213 (IO)
- net A24: now also U18.207 (IO)
- net A25: now also U18.208 (IO)
- net A26: now also U18.204 (IO)
- net A27: now also U18.206 (IO)
- net A28: now also U18.201 (IO)
- net A29: now also U18.202 (IO)
- net A3: now also U18.236 (IO)
- net A30: now also U18.198 (IO)
- net A31: now also U18.199 (IO)
- net A4: now also U18.234 (IO)
- net A5: now also U18.233 (IO)
- net A6: now also U18.235 (IO)
- net A7: now also U18.228 (IO)
- net A8: now also U18.227 (IO)
- net A9: now also U18.232 (IO)
- net D0: now also U18.8 (IO)
- net D1: now also U18.36 (IO)
- net D10: now also U18.38 (IO)
- net D11: now also U18.37 (IO)
- net D12: now also U18.40 (IO)
- net D13: now also U18.39 (IO)
- net D14: now also U18.41 (IO)
- net D15: now also U18.18 (IO)
- net D16: now also U18.19 (IO)
- net D17: now also U18.42 (IO)
- net D18: now also U18.20 (IO)
- net D19: now also U18.43 (IO)
- net D2: now also U18.15 (IO)
- net D20: now also U18.27 (IO)
- net D21: now also U18.46 (IO)
- net D22: now also U18.45 (IO)
- net D23: now also U18.47 (IO)
- net D24: now also U18.48 (IO)
- net D25: now also U18.53 (IO)
- net D26: now also U18.55 (IO)
- net D27: now also U18.56 (IO)
- net D28: now also U18.57 (IO)
- net D29: now also U18.58 (IO)
- net D3: now also U18.17 (IO)
- net D30: now also U18.59 (IO)
- net D31: now also U18.60 (IO)
- net D4: now also U18.14 (IO)
- net D5: now also U18.33 (IO)
- net D6: now also U18.16 (IO)
- net D7: now also U18.13 (IO)
- net D8: now also U18.34 (IO)
- net D9: now also U18.35 (IO)
- net FC0: now also U18.185 (IO)
- net FC1: now also U18.187 (IO)
- net FC2: now also U18.183 (IO)
- net R/~{W}: now also U18.21 (IO)
- net SIZ0: now also U18.6 (IO)
- net SIZ1: now also U18.7 (IO)
- net ~{AS}: now also U18.4 (IO)
- net ~{BERR}: now also U18.182 (IO)
- net ~{BGACK}: now also U18.196 (IO)
- net ~{BG}: now also U18.194 (IO)
- net ~{BR}: now also U18.190 (IO)
- net ~{CBACK}: now also U18.26 (IO)
- net ~{CBREQ}: now also U18.25 (IO)
- net ~{CDIS}: now also U18.2 (IO)
- net ~{CIIN}: now also U18.193 (IO)
- net ~{CIOUT}: now also U18.24 (IO)
- net ~{DS}: now also U18.5 (IO)
- net ~{IPL0}: now also U18.3 (IO)
- net ~{IPL1}: now also U18.239 (IO)
- net ~{IPL2}: now also U18.1 (IO)
- net ~{RMC}: now also U18.189 (IO)
- net ~{STERM}: now also U18.238 (IO)
- new net CACHE_TD0: U18.140 (IO)
- new net CACHE_TD1: U18.139 (IO)
- new net CACHE_TD10: U18.127 (IO)
- new net CACHE_TD11: U18.126 (IO)
- new net CACHE_TD12: U18.125 (IO)
- new net CACHE_TD13: U18.123 (IO)
- new net CACHE_TD14: U18.122 (IO)
- new net CACHE_TD15: U18.121 (IO)
- new net CACHE_TD2: U18.138 (IO)
- new net CACHE_TD3: U18.137 (IO)
- new net CACHE_TD4: U18.136 (IO)
- new net CACHE_TD5: U18.135 (IO)
- new net CACHE_TD6: U18.134 (IO)
- new net CACHE_TD7: U18.133 (IO)
- new net CACHE_TD8: U18.132 (IO)
- new net CACHE_TD9: U18.128 (IO)
- new net SIMM_PDQ0: U18.179 (IO)
- new net SIMM_PDQ1: U18.177 (IO)
- new net SIMM_PDQ2: U18.178 (IO)
- new net SIMM_PDQ3: U18.180 (IO)
- new net SIMM_SA0: U18.145 (IO)
- new net SIMM_SA1: U18.146 (IO)
- new net SIMM_SA10: U18.158 (IO)
- new net SIMM_SA11: U18.168 (IO)
- new net SIMM_SA2: U18.147 (IO)
- new net SIMM_SA3: U18.153 (IO)
- new net SIMM_SA4: U18.154 (IO)
- new net SIMM_SA5: U18.156 (IO)
- new net SIMM_SA6: U18.157 (IO)
- new net SIMM_SA7: U18.167 (IO)
- new net SIMM_SA8: U18.173 (IO)
- new net SIMM_SA9: U18.174 (IO)
- new net SIMM_~{CAS0}: U18.141 (IO)
- new net SIMM_~{CAS1}: U18.144 (IO)
- new net SIMM_~{CAS2}: U18.142 (IO)
- new net SIMM_~{CAS3}: U18.143 (IO)
- new net SIMM_~{RAS0}: U18.160 (IO)
- new net SIMM_~{RAS1}: U18.159 (IO)
- new net SIMM_~{RAS2}: U18.163 (IO)
- new net SIMM_~{RAS3}: U18.162 (IO)
- new net SIMM_~{RAS4}: U18.165 (IO)
- new net SIMM_~{RAS5}: U18.164 (IO)
- new net SIMM_~{RAS6}: U18.176 (IO)
- new net SIMM_~{RAS7}: U18.175 (IO)
Other:
- note removed: "Local Bus Signals"
