File: kicad/projects/m68k-hbc/SBC.kicad_sch (KiCad schematic)
At the start: 19 parts, among them U8 SBC

Commit message: Large changes: EHBCSimpleEmu, kicad, fwcode, docs
This commit contains some large changes:
- Removed EHBCSimpleEmu (Moved to kms1212/llemu, kms1212/qemu)
- (likely) Removed fwcode; now it only boots and stops
- Modified documents
Parts:
- removed C163, C164, C165, C166, C167, C168, C18, C19, C20, C21, C22, C23, C24, C25, C26, C27, C28, C29: C, Capacitor_SMD:C_0603_1608Metric_Pad1.08x0.95mm_HandSolder, symbol Device:C
- added unit 2 of U8
- U8: value SBC -> EPF6016QC240
Connections:
- net A0: no longer U8.125 (IO)
- net A1: no longer U8.126 (IO)
- net A10: no longer U8.138 (IO)
- net A11: no longer U8.139 (IO)
- net A12: no longer U8.140 (IO)
- net A13: no longer U8.141 (IO)
- net A14: no longer U8.142 (IO)
- net A15: no longer U8.143 (IO)
- net A2: no longer U8.127 (IO)
- net A3: no longer U8.128 (IO)
- net A4: no longer U8.132 (IO)
- net A5: no longer U8.133 (IO)
- net A6: no longer U8.134 (IO)
- net A7: no longer U8.135 (IO)
- net A8: no longer U8.136 (IO)
- net A9: no longer U8.137 (IO)
- net D0: no longer U8.84 (IO)
- net D1: no longer U8.85 (IO)
- net D10: no longer U8.98 (IO)
- net D11: no longer U8.99 (IO)
- net D12: no longer U8.100 (IO)
- net D13: no longer U8.101 (IO)
- net D14: no longer U8.102 (IO)
- net D15: no longer U8.103 (IO)
- net D16: no longer U8.104 (IO)
- net D17: no longer U8.105 (IO)
- net D18: no longer U8.106 (IO)
- net D19: no longer U8.107 (IO)
- net D2: no longer U8.86 (IO)
- net D20: no longer U8.108 (IO)
- net D21: no longer U8.111 (IO)
- net D22: no longer U8.112 (IO)
- net D23: no longer U8.113 (IO)
- net D24: no longer U8.114 (IO)
- net D25: no longer U8.115 (IO)
- net D26: no longer U8.116 (IO)
- net D27: no longer U8.118 (IO)
- net D28: no longer U8.119 (IO)
- net D29: no longer U8.121 (IO)
- net D3: no longer U8.87 (IO)
- net D30: no longer U8.122 (IO)
- net D31: no longer U8.123 (IO)
- net D4: no longer U8.88 (IO)
- net D5: no longer U8.93 (IO)
- net D6: no longer U8.94 (IO)
- net D7: no longer U8.95 (IO)
- net D8: no longer U8.96 (IO)
- net D9: no longer U8.97 (IO)
- net ISA_A16: no longer U8.42 (IO)
- net ISA_A17: no longer U8.41 (IO)
- net ISA_A18: no longer U8.40 (IO)
- net ISA_A19: no longer U8.39 (IO)
- net AD0: no longer names the net of U8.43 (IO)
- net AD1: no longer names the net of U8.45 (IO)
- net AD10: no longer names the net of U8.59 (IO)
- net AD11: no longer names the net of U8.60 (IO)
- net AD12: no longer names the net of U8.62 (IO)
- net AD13: no longer names the net of U8.63 (IO)
- net AD14: no longer names the net of U8.64 (IO)
- net AD15: no longer names the net of U8.65 (IO)
- net AD16: no longer names the net of U8.66 (IO)
- net AD17: no longer names the net of U8.67 (IO)
- net AD18: no longer names the net of U8.68 (IO)
- net AD19: no longer names the net of U8.69 (IO)
- net AD2: no longer names the net of U8.46 (IO)
- net AD20: no longer names the net of U8.70 (IO)
- net AD21: no longer names the net of U8.73 (IO)
- net AD22: no longer names the net of U8.74 (IO)
- net AD23: no longer names the net of U8.75 (IO)
- net AD24: no longer names the net of U8.76 (IO)
- net AD25: no longer names the net of U8.77 (IO)
- net AD26: no longer names the net of U8.78 (IO)
- net AD27: no longer names the net of U8.79 (IO)
- net AD28: no longer names the net of U8.80 (IO)
- net AD29: no longer names the net of U8.81 (IO)
- net AD3: no longer names the net of U8.47 (IO)
- net AD30: no longer names the net of U8.82 (IO)
- net AD31: no longer names the net of U8.83 (IO)
- net AD4: no longer names the net of U8.48 (IO)
- net AD5: no longer names the net of U8.53 (IO)
- net AD6: no longer names the net of U8.55 (IO)
- net AD7: no longer names the net of U8.56 (IO)
- net AD8: no longer names the net of U8.57 (IO)
- net AD9: no longer names the net of U8.58 (IO)
- net ISACLK: no longer names the net of U8.157 (IO)
- net ISA_LA17: no longer names the net of U8.38 (IO)
- net PEPCLK: no longer names the net of U8.158 (IO)
- net REFCLK: no longer names the net of U8.156 (IO)
- net R/~{W}: no longer names the net of U8.146 (IO)
- net SB37: no longer names the net of U8.37 (IO)
- net SB38: no longer names the net of U8.36 (IO)
- net SB39: no longer names the net of U8.35 (IO)
- net SB40: no longer names the net of U8.34 (IO)
- net SB41: no longer names the net of U8.33 (IO)
- net SB42: no longer names the net of U8.27 (IO)
- net SBCDCL: no longer names the net of U8.165 (IO)
- net ~{AS}: no longer names the net of U8.144 (IO)
- net ~{CS_SBC}: no longer names the net of U8.167 (IO)
- net ~{DS}: no longer names the net of U8.145 (IO)
- net ~{IACK}: no longer names the net of U8.162 (IO)
- net ~{IRQ_SBC}: no longer names the net of U8.160 (IO)
- net ~{RST_SBC}: no longer names the net of U8.159 (IO)
- net ~{SBCDACK}: no longer names the net of U8.164 (IO)
- net ~{SBCDRQ}: no longer names the net of U8.163 (IO)
- net ~{STERM}: no longer names the net of U8.147 (IO)
Other:
- note removed: "ATA Signals"
- note removed: "ISA Signals"
- note removed: "Local Bus Signals"
- note removed: "OPB Signals"
- note removed: "PEP Signals"
