File: kicad/projects/m68k-hbc/m68k-hbc.kicad_pcb (KiCad board)
At the start: 6 copper layers, 304.8 x 243.8 mm, 218 parts, among them IC1 MC68030RC, IC2 MC68881FN, J1 JTAG_DRAMC, J10 ATX-24, J11 Conn_02x12_Odd_Even, J12 ICSP_SMC, J13 IDC_PATA, J14 IDC_FDD, J15 5747840-4, J16 KMDGX-6SG_P-S4N, J17 RJ45_Amphenol_RJMG1BD3B8K1ANR, J18 JTAG_PIC, J19 JTAG_ADDEC, J2 PEP_Power_DIN41612_3x10, J3 PEP_Power_DIN41612_3x10, J4 PEP_Power_DIN41612_3x10, J5 PEP_Data_DIN41612_3x32, J6 PEP_Data_DIN41612_3x32, J7 PEP_Data_DIN41612_3x32, J8 Bus_ISA_16bit, J9 Bus_ISA_16bit, U1 SIMM72 Slot A, U10 74LS245, U11 MCP23017_SO, U12 MCP23017_SO, U13 74LS02, U14 25LCxxx, U15 DS1307+, U16 ATmegA32-16P, U17 PCA9306D, U18 74LS137, U18 SN74LV1T34DBV, U19 Si5351A-B-GT, U2 SIMM72 Slot B, U20 SN74LV1T34DBV, U21 SN74LV1T34DBV, U22 PC8477BV, U23 MAX232, U24 68681, U25 68230, U26 74LS06, U27 VT82C42, U28 FWMC, U29 RTL8019AS, U3 SIMM72 Slot C, U30 EPM7128SLC84 / Programmable I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, U31 74LS04, U32 74LS245, U33 74LS573, U34 MC68440FN, U35 74LS245, U36 74LS245, U37 74LS573, U38 74LS137, U39 EPM7128SLC84 / Address Decoder, U4 SIMM72 Slot D, U40 74LS137, U41 74LS139, U42 74LS137, U5 EPM7128SLC84 / DRAM Controller, U6 74LS137, U7 74LS245, U8 74LS245, U9 74LS245, X1 70M, X2 8M, X3 70M, X4 10M, X5 70M, Y1 32.768k, Y2 16M, Y3 25M, Y4 24M, Y5 3.6864M, Y6 8M, Y7 20M

Commit message: Modified system architecture, New KiCad Project: Cache Memory Module(SIMM80)
Parts:
- removed the C1 at (139.7, 144.2)
- removed the C10 at (111.1, 123.5)
- removed the C11 at (125.1, 123.5)
- removed the C12 at (137.8, 123.5)
- removed the C13 at (151.8, 123.5)
- removed the C14 at (111.1, 64.8)
- removed the C2 at (144.7, 142.9)
- removed the C3 at (139.7, 161.9)
- removed the C32 at (308.2, 146.1)
- removed the C33 at (300.6, 154.9)
- removed the C39 at (199.7, 57.1)
- removed the C39 at (174.6, 123.5)
- removed the C4 at (144.7, 163.2)
- removed the C45 at (136.2, 187.3)
- removed the C46 at (131.1, 187.3)
- removed the C5 at (152.3, 163.2)
- removed the C53 at (107.7, 209.6)
- removed the C54 at (117.4, 240.7)
- removed the C55 at (117.8, 257.2)
- removed the C56 at (123.8, 256.2)
- removed the C57 at (120.3, 231.1)
- removed the C58 at (120.3, 227.3)
- removed the C59 at (116.2, 254.6)
- removed the C6 at (160.0, 161.9)
- removed the C60 at (128.9, 256.2)
- removed the C61 at (80.6, 165.1)
- removed the C7 at (157.4, 142.9)
- removed the C8 at (160.0, 146.7)
- removed the C9 at (95.9, 123.5)
- removed the J1 at (172.7, 137.2)
- removed the J15 at (97.7, 270.2)
- removed the R1 at (227.7, 64.1)
- removed REF**: IDC-Header_2x32_P2.54mm_Vertical, Connector_IDC:IDC-Header_2x32_P2.54mm_Vertical
- removed RN10: 1k, Resistor_THT:R_Array_SIP6
- removed the RN5 at (180.9, 147.3)
- removed U1: SIMM72 Slot A, Sockets:SIM72
- removed the U10 at (95.9, 123.4)
- removed the U11 at (108.6, 62.9)
- removed the U12 at (300.6, 139.1)
- removed the U13 at (300.6, 154.9)
- removed the U15 at (304.8, 91.4)
- removed the U18 at (137.8, 123.6)
- removed the U18 at (126.7, 176.7)
- removed U2: SIMM72 Slot B, Sockets:SIM72
- removed the U3 at (132.7, 100.3)
- removed the U4 at (132.7, 113.0)
- removed the U5 at (149.8, 137.8)
- removed the U6 at (125.1, 123.6)
- removed the U8 at (151.8, 123.4)
- removed the U9 at (111.1, 123.4)
- removed X4: 10M, Oscillator:Oscillator_SMD_SeikoEpson_SG8002CA-4Pin_7.0x5.0mm
- removed X5: 70M, Oscillator:Oscillator_SMD_SeikoEpson_SG8002CA-4Pin_7.0x5.0mm
- removed the Y1 at (304.8, 95.2)
- removed the Y3 at (131.5, 183.5)
- added C100: 33p, Capacitor_SMD:C_1206_3216Metric_Pad1.33x1.80mm_HandSolder, F.Cu at (138.1, 211.5)
- added C101: 10u, Capacitor_THT:CP_Radial_D5.0mm_P2.50mm, F.Cu at (150.4, 274.3)
- added C102: 33p, Capacitor_SMD:C_1206_3216Metric_Pad1.33x1.80mm_HandSolder, F.Cu at (138.1, 221.6)
- added C103: 47p, Capacitor_SMD:C_1206_3216Metric_Pad1.33x1.80mm_HandSolder, F.Cu at (149.8, 252.4)
- added C104: 1.2n, Capacitor_SMD:C_1206_3216Metric_Pad1.33x1.80mm_HandSolder, F.Cu at (149.8, 268.3)
- added C105: 100n, Capacitor_SMD:C_1206_3216Metric_Pad1.33x1.80mm_HandSolder, B.Cu at (142.8, 267.3)
- added C106: 33p, Capacitor_SMD:C_1206_3216Metric_Pad1.33x1.80mm_HandSolder, F.Cu at (138.1, 226.7)
- added C107: 100n, Capacitor_SMD:C_1206_3216Metric_Pad1.33x1.80mm_HandSolder, B.Cu at (142.8, 251.5)
- added C108: 47p, Capacitor_SMD:C_1206_3216Metric_Pad1.33x1.80mm_HandSolder, F.Cu at (132.6, 246.4)
- added C109: 10u, Capacitor_THT:CP_Radial_D5.0mm_P2.50mm, F.Cu at (132.7, 238.1)
- added C110: 1.8n, Capacitor_SMD:C_1206_3216Metric_Pad1.33x1.80mm_HandSolder, F.Cu at (141.9, 232.4)
- added C111: 1u, Capacitor_SMD:C_1206_3216Metric_Pad1.33x1.80mm_HandSolder, F.Cu at (157.2, 236.9)
- added C112: 1u, Capacitor_SMD:C_1206_3216Metric_Pad1.33x1.80mm_HandSolder, F.Cu at (157.2, 239.4)
- added C113: 10u, Capacitor_THT:CP_Radial_D5.0mm_P2.50mm, F.Cu at (150.4, 238.1)
- added C114: 1.8n, Capacitor_SMD:C_1206_3216Metric_Pad1.33x1.80mm_HandSolder, F.Cu at (133.6, 232.4)
- added C115: 47p, Capacitor_SMD:C_1206_3216Metric_Pad1.33x1.80mm_HandSolder, F.Cu at (153.0, 246.4)
- added C116: 100n, Capacitor_SMD:C_1210_3225Metric, B.Cu at (142.8, 237.5)
- added C117: 100n, Capacitor_SMD:C_1206_3216Metric_Pad1.33x1.80mm_HandSolder, B.Cu at (188.7, 248.9)
- added C118: 100n, Capacitor_SMD:C_1206_3216Metric_Pad1.33x1.80mm_HandSolder, B.Cu at (186.2, 245.1)
- added C119: 100n, Capacitor_SMD:C_1206_3216Metric_Pad1.33x1.80mm_HandSolder, B.Cu at (190.6, 245.1)
- added C120: 1u, Capacitor_SMD:C_1206_3216Metric_Pad1.33x1.80mm_HandSolder, B.Cu at (184.8, 266.1)
- added C121: 4.7u, Capacitor_SMD:C_1206_3216Metric_Pad1.33x1.80mm_HandSolder, B.Cu at (184.8, 273.1)
- added C122: 10p, Capacitor_SMD:C_1206_3216Metric_Pad1.33x1.80mm_HandSolder, F.Cu at (192.4, 253.7)
- added C123: 22p, Capacitor_SMD:C_1206_3216Metric_Pad1.33x1.80mm_HandSolder, F.Cu at (200.0, 253.7)
- added C124: 22p, Capacitor_SMD:C_1206_3216Metric_Pad1.33x1.80mm_HandSolder, F.Cu at (194.9, 253.7)
- added C125: 22p, Capacitor_SMD:C_1206_3216Metric_Pad1.33x1.80mm_HandSolder, F.Cu at (175.0, 148.0)
- added C126: 22p, Capacitor_SMD:C_1206_3216Metric_Pad1.33x1.80mm_HandSolder, F.Cu at (170.0, 148.0)
- added C127: 100n, Capacitor_SMD:C_1206_3216Metric_Pad1.33x1.80mm_HandSolder, F.Cu at (-53.4, 144.1)
- added C128: 100n, Capacitor_SMD:C_1206_3216Metric_Pad1.33x1.80mm_HandSolder, F.Cu at (-53.4, 147.5)
- added C129: 100n, Capacitor_SMD:C_1206_3216Metric_Pad1.33x1.80mm_HandSolder, F.Cu at (-53.4, 150.8)
- added C130: 100n, Capacitor_SMD:C_1206_3216Metric_Pad1.33x1.80mm_HandSolder, F.Cu at (-53.4, 154.2)
- added C131: 100n, Capacitor_SMD:C_1206_3216Metric_Pad1.33x1.80mm_HandSolder, F.Cu at (-53.4, 157.5)
- added C132: 100n, Capacitor_SMD:C_1206_3216Metric_Pad1.33x1.80mm_HandSolder, F.Cu at (-65.4, 150.8)
- added C133: 100n, Capacitor_SMD:C_1206_3216Metric_Pad1.33x1.80mm_HandSolder, F.Cu at (-65.4, 154.2)
- added C134: 100n, Capacitor_SMD:C_1206_3216Metric_Pad1.33x1.80mm_HandSolder, F.Cu at (-65.4, 157.5)
- added C135: 100n, Capacitor_SMD:C_1206_3216Metric_Pad1.33x1.80mm_HandSolder, F.Cu at (-59.4, 144.1)
- added C136: 100n, Capacitor_SMD:C_1206_3216Metric_Pad1.33x1.80mm_HandSolder, F.Cu at (-59.4, 147.5)
- added C137: 100n, Capacitor_SMD:C_1206_3216Metric_Pad1.33x1.80mm_HandSolder, F.Cu at (-59.4, 150.8)
- added C138: 100n, Capacitor_SMD:C_1206_3216Metric_Pad1.33x1.80mm_HandSolder, F.Cu at (-65.4, 144.1)
- added C139: 100n, Capacitor_SMD:C_1206_3216Metric_Pad1.33x1.80mm_HandSolder, F.Cu at (-65.4, 147.5)
- added C140: 100n, Capacitor_SMD:C_1206_3216Metric_Pad1.33x1.80mm_HandSolder, F.Cu at (-59.4, 154.2)
- added C141: 100n, Capacitor_SMD:C_1206_3216Metric_Pad1.33x1.80mm_HandSolder, F.Cu at (-59.4, 157.5)
- added C148: 1m, Capacitor_THT:CP_Radial_D8.0mm_P3.50mm, F.Cu at (68.9, 143.5)
- added C149: 1m, Capacitor_THT:CP_Radial_D8.0mm_P3.50mm, F.Cu at (68.9, 152.4)
- added C18: 1m, Capacitor_THT:CP_Radial_D8.0mm_P3.50mm, F.Cu at (83.8, 128.3)
- added C19: 1m, Capacitor_THT:CP_Radial_D8.0mm_P3.50mm, F.Cu at (83.8, 137.2)
- added C37: 100n, Capacitor_SMD:C_1206_3216Metric_Pad1.33x1.80mm_HandSolder, B.Cu at (106.7, 182.2)
- added C39: 1u, Capacitor_SMD:C_1206_3216Metric_Pad1.33x1.80mm_HandSolder, F.Cu at (88.9, 249.2)
- added C40: 1u, Capacitor_SMD:C_1206_3216Metric_Pad1.33x1.80mm_HandSolder, F.Cu at (90.5, 255.3)
- added C41: 1u, Capacitor_SMD:C_1206_3216Metric_Pad1.33x1.80mm_HandSolder, F.Cu at (92.1, 247.7)
- added C42: 1u, Capacitor_SMD:C_1206_3216Metric_Pad1.33x1.80mm_HandSolder, F.Cu at (90.5, 260.4)
- added C77: 1.2n, Capacitor_SMD:C_1206_3216Metric_Pad1.33x1.80mm_HandSolder, F.Cu at (133.3, 263.2)
- added C78: 47p, Capacitor_SMD:C_1206_3216Metric_Pad1.33x1.80mm_HandSolder, F.Cu at (135.8, 252.4)
- added C79: 100n, Capacitor_SMD:C_1206_3216Metric_Pad1.33x1.80mm_HandSolder, B.Cu at (160.4, 210.2)
- added C80: 100n, Capacitor_SMD:C_1206_3216Metric_Pad1.33x1.80mm_HandSolder, B.Cu at (154.0, 210.2)
- added C81: 1u, Capacitor_THT:CP_Radial_D5.0mm_P2.50mm, F.Cu at (136.6, 205.7)
- added C82: 1u, Capacitor_THT:CP_Radial_D5.0mm_P2.50mm, F.Cu at (140.4, 200.7)
- added C83: 100n, Capacitor_SMD:C_1206_3216Metric_Pad1.33x1.80mm_HandSolder, B.Cu at (152.7, 214.0)
- added C91: 1u, Capacitor_SMD:C_1206_3216Metric_Pad1.33x1.80mm_HandSolder, F.Cu at (140.3, 248.3)
- added C92: 1u, Capacitor_THT:CP_Radial_D5.0mm_P2.50mm, F.Cu at (158.0, 251.3)
- added C93: 1u, Capacitor_THT:CP_Radial_D5.0mm_P2.50mm, F.Cu at (167.5, 246.2)
- added C94: 470n, Capacitor_SMD:C_1206_3216Metric_Pad1.33x1.80mm_HandSolder, F.Cu at (162.9, 239.4)
- added C95: 33p, Capacitor_SMD:C_1206_3216Metric_Pad1.33x1.80mm_HandSolder, F.Cu at (138.1, 216.5)
- added C96: 1u, Capacitor_THT:CP_Radial_D5.0mm_P2.50mm, F.Cu at (170.7, 251.3)
- added C97: 1u, Capacitor_THT:CP_Radial_D5.0mm_P2.50mm, F.Cu at (161.2, 246.2)
- added C98: 1u, Capacitor_SMD:C_1206_3216Metric_Pad1.33x1.80mm_HandSolder, F.Cu at (149.8, 263.2)
- added C99: 1u, Capacitor_SMD:C_1206_3216Metric_Pad1.33x1.80mm_HandSolder, F.Cu at (145.3, 248.3)
- added D1: D, Diode_THT:D_5W_P10.16mm_Horizontal, F.Cu at (68.6, 135.9)
- added D3: D, Diode_THT:D_5W_P10.16mm_Horizontal, F.Cu at (77.5, 144.4)
- added FB2: FerriteBead, Inductor_THT:L_Axial_L5.0mm_D3.6mm_P10.00mm_Horizontal_Murata_BL01RN1A2A2, F.Cu at (236.9, 277.5)
- added FB3: FerriteBead, Inductor_THT:L_Axial_L5.3mm_D2.2mm_P2.54mm_Vertical_Vishay_IM-1, F.Cu at (142.2, 207.6)
- added IC3: MC68901P, Package_DIP:DIP-48_W15.24mm_Socket, F.Cu at (110.5, 205.7)
- added J14: 5747840-4, 57478404:57478404, F.Cu at (97.8, 271.0)
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- renumbered C34 to C22, C35 to C23, C36 to C24, C37 to C25, C40 to C26, C41 to C27, C43 to C29, C44 to C30, C51 to C35, C52 to C36, C64 to C45, C65 to C46, C66 to C47, C67 to C48, C68 to C49, C69 to C50, C70 to C51, C71 to C52, C72 to C53, C73 to C54, C74 to C55, C75 to C56, D1 to D2, H6 to H10, H7 to H11, H8 to H12, H9 to H13, J2 to J1, J12 to J10, J13 to J12, J14 to J13, J16 to J15, J17 to J16, J18 to J17, J19 to J18, J3 to J2, J4 to J3, J5 to J4, J6 to J5, J7 to J6, J8 to J7, J9 to J8, J10 to J9, R2 to R1, R9 to R10, R10 to R11, R3 to R2, R4 to R5, R5 to R6, R6 to R7, R7 to R8, R8 to R9, RN6 to RN1, RN7 to RN2, RN8 to RN3, RN9 to RN4, RN11 to RN5, U28 to U10, U29 to U11, U30 to U12, U38 to U13, U39 to U14, U40 to U15, U41 to U16, U42 to U17, U14 to U3, U16 to U4, U17 to U5, U22 to U6, U26 to U8, U27 to U9, Y2 to Y1, Y4 to Y2, Y6 to Y3, Y7 to Y4
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Connections:
- net /SMC/~{DTACK} renamed /SMC/~{DTACK8}
- net ~{ATADRQ} renamed ATADRQ
- net ~{ATAIRQ} renamed ATAIRQ
- C1 pad 1: +5V -> CPUPWR
- C10 pad 2: +5V -> CPUPWR
- C11 pad 2: +5V -> CPUPWR
- C12 pad 1: +5V -> CPUPWR
- C13 pad 1: +5V -> CPUPWR
- C14 pad 1: +5V -> CPUPWR
- C15 pad 2: +5V -> CPUPWR
- C16 pad 1: +5V -> CPUPWR
- C17 pad 1: +5V -> CPUPWR
- C2 pad 1: +5V -> CPUPWR
- C22 pad 1: /Power/+12VI -> +12V
- C24 pad 1: /Power/+5VI -> +5V
- C26 pad 1: /Power/+3.3VI -> +3.3V
- C3 pad 2: +5V -> CPUPWR
- C38 pad 1: /Power/+5VSBI -> +5V
- C4 pad 1: +5V -> CPUPWR
- C5 pad 2: +5V -> CPUPWR
- C6 pad 1: +5V -> CPUPWR
- C7 pad 1: +5V -> CPUPWR
- C8 pad 1: +5V -> CPUPWR
- C84 pad 1: +5V -> /Audio/VD34
- C84 pad 2: GND -> GNDA
- C85 pad 1: +5V -> +5VA
- C85 pad 2: GND -> GNDA
- C86 pad 1: +5V -> +5VA
- C86 pad 2: GND -> GNDA
- C87 pad 1: +5V -> Net-(C87-Pad1)
- C87 pad 2: GND -> GNDA
- C88 pad 1: +5V -> Net-(U20-VREFI)
- C88 pad 2: GND -> GNDA
- C89 pad 1: +5V -> Net-(U20-VREFI)
- C89 pad 2: GND -> GNDA
- C9 pad 1: +5V -> CPUPWR
- C90 pad 1: GND -> Net-(C77-Pad2)
- C90 pad 2: +5V -> /Audio/LMIC
- H1 pad 1: GND -> GNDPWR
- H10 pad 1: GND -> GNDPWR
- H11 pad 1: GND -> GNDPWR
- H12 pad 1: GND -> GNDPWR
- H13 pad 1: GND -> GNDPWR
- H2 pad 1: GND -> GNDPWR
- H3 pad 1: GND -> GNDPWR
- H4 pad 1: GND -> GNDPWR
- H5 pad 1: GND -> GNDPWR
- IC1 pad C06: +5V -> CPUPWR
- IC1 pad D04: +5V -> CPUPWR
- IC1 pad D10: +5V -> CPUPWR
- IC1 pad F02: +5V -> CPUPWR
- IC1 pad F11: +5V -> CPUPWR
- IC1 pad H03: +5V -> CPUPWR
- IC1 pad H11: +5V -> CPUPWR
- IC1 pad K04: +5V -> CPUPWR
- IC1 pad K10: +5V -> CPUPWR
- IC1 pad L06: +5V -> CPUPWR
- IC2 pad 10: +5V -> CPUPWR
- IC2 pad 16: +5V -> CPUPWR
- IC2 pad 17: +5V -> CPUPWR
- IC2 pad 27: +5V -> CPUPWR
- IC2 pad 43: +5V -> CPUPWR
- IC2 pad 52: +5V -> CPUPWR
- IC2 pad 53: +5V -> CPUPWR
- IC2 pad 61: +5V -> CPUPWR
- J11 pad 1: unconnected-(J11-Pin_1-Pad1) -> GND
- J11 pad 3: unconnected-(J11-Pin_3-Pad3) -> SMC_TX
- J11 pad 5: unconnected-(J11-Pin_5-Pad5) -> SMC_RX
- J11 pad 7: unconnected-(J11-Pin_7-Pad7) -> GND
- J12 pad 39: unconnected-(J13-~{LED}-Pad39) -> Net-(J12-~{LED})
- J15 pad MH1: GND -> GNDPWR
- J15 pad MH2: GND -> GNDPWR
- J15 pad MH3: GND -> GNDPWR
- J15 pad MH4: GND -> GNDPWR
- J15 pad MH5: GND -> GNDPWR
- J16 pad 13: GND -> GNDPWR
- J9 pad 1: /Power/+3.3VI -> +3.3V
- J9 pad 10: /Power/+12VI -> +12V
- J9 pad 11: /Power/+12VI -> +12V
- J9 pad 12: /Power/+3.3VI -> +3.3V
- J9 pad 13: /Power/+3.3VI -> +3.3V
- J9 pad 2: /Power/+3.3VI -> +3.3V
- J9 pad 21: /Power/+5VI -> +5V
- J9 pad 22: /Power/+5VI -> +5V
- J9 pad 23: /Power/+5VI -> +5V
- J9 pad 4: /Power/+5VI -> +5V
- J9 pad 6: /Power/+5VI -> +5V
- J9 pad 9: /Power/+5VSBI -> +5VP
- L1 pad 1: /Power/+12VI -> +5V
- L1 pad 2: +12V -> CPUPWR
- L2 pad 1: /Power/+5VI -> /Audio/PINKTIP
- L2 pad 2: +5V -> Net-(C92-Pad1)
- L3 pad 1: /Power/+5VSBI -> /Audio/BLUERING
- L3 pad 2: +5VP -> Net-(C93-Pad1)
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Other:
- board text added: "68k30 HBC Motherboard"
- board text added: "ATX-Size 12inx9.6in"
- board text added: "Designed by kms1212(Minsu Kwon)"
- board text added: "Rev.1 2023/xx/xx"

Commit message: Some Updates
Parts:
- removed the RN1 at (68.6, 70.8)
- removed the RN1 at (355.6, 49.5)
- removed the RN2 at (354.3, 83.8)
- removed the RN2 at (72.4, 80.9)
- removed the RN3 at (221.0, 278.1)
- removed the RN3 at (68.6, 91.1)
- removed the RN4 at (72.4, 101.3)
- removed the RN4 at (301.0, 67.3)
- removed RN7: 10k, Resistor_THT:R_Array_SIP9
- removed the U30 at (209.6, 170.2)
- removed the U30 at (241.3, 62.2)
- removed U41, U42, U45, U46, U49, U50: 74LS245, Package_SO:SOP-20_7.5x12.8mm_P1.27mm
- removed U43, U51: MC74LCX16245DT, Package_SO:TSSOP-48_6.1x12.5mm_P0.5mm
- removed X3: 4M, Oscillator:Oscillator_SMD_SeikoEpson_SG8002CA-4Pin_7.0x5.0mm
- removed Y9: 25M, Crystal:Crystal_HC52-6mm_Vertical
- added C142: 150u, Capacitor_THT:CP_Radial_D5.0mm_P2.50mm, F.Cu at (-18.5, 324.7)
- added C143: 22u, Capacitor_SMD:C_0603_1608Metric_Pad1.08x0.95mm_HandSolder, F.Cu at (-9.03, 290.1)
- added C144: 22u, Capacitor_SMD:C_0603_1608Metric_Pad1.08x0.95mm_HandSolder, F.Cu at (-9.03, 292.6)
- added C145: 22u, Capacitor_SMD:C_0603_1608Metric_Pad1.08x0.95mm_HandSolder, F.Cu at (-9.03, 295.1)
- added C146: 22u, Capacitor_SMD:C_0603_1608Metric_Pad1.08x0.95mm_HandSolder, F.Cu at (-9.03, 297.6)
- added C147: 470u, Capacitor_THT:CP_Radial_D8.0mm_P3.50mm, F.Cu at (-48.3, 278.0)
- added C150: 47u, Capacitor_THT:CP_Radial_D8.0mm_P3.50mm, F.Cu at (-48.3, 306.7)
- added C151: 150u, Capacitor_THT:CP_Radial_D5.0mm_P2.50mm, F.Cu at (-18.5, 331.2)
- added C152: 150u, Capacitor_THT:CP_Radial_D5.0mm_P2.50mm, F.Cu at (-18.5, 337.8)
- added C153: 22u, Capacitor_SMD:C_0603_1608Metric_Pad1.08x0.95mm_HandSolder, F.Cu at (-9.03, 300.1)
- added C154: 22u, Capacitor_SMD:C_0603_1608Metric_Pad1.08x0.95mm_HandSolder, F.Cu at (-9.03, 302.6)
- added C155: 22u, Capacitor_SMD:C_0603_1608Metric_Pad1.08x0.95mm_HandSolder, F.Cu at (-9.03, 305.1)
- added C156: 22u, Capacitor_SMD:C_0603_1608Metric_Pad1.08x0.95mm_HandSolder, F.Cu at (-9.03, 307.6)
- added C157: 10u, Capacitor_SMD:C_0603_1608Metric_Pad1.08x0.95mm_HandSolder, F.Cu at (-9.03, 310.1)
- added C158: 100n, Capacitor_SMD:C_0603_1608Metric_Pad1.08x0.95mm_HandSolder, F.Cu at (-4.68, 287.5)
- added C159: 1u, Capacitor_SMD:C_0603_1608Metric_Pad1.08x0.95mm_HandSolder, F.Cu at (-4.68, 290.1)
- added C160: 470u, Capacitor_THT:CP_Radial_D8.0mm_P3.50mm, F.Cu at (-48.3, 316.2)
- added C161: 47u, Capacitor_THT:CP_Radial_D8.0mm_P3.50mm, F.Cu at (-48.3, 325.8)
- added C162: 100n, Capacitor_SMD:C_0603_1608Metric_Pad1.08x0.95mm_HandSolder, F.Cu at (-4.68, 292.6)
- added C163: 100n, Capacitor_SMD:C_0603_1608Metric_Pad1.08x0.95mm_HandSolder, F.Cu at (-4.68, 295.1)
- added C164: 1u, Capacitor_SMD:C_0603_1608Metric_Pad1.08x0.95mm_HandSolder, F.Cu at (-4.68, 297.6)
- added C165: 1u, Capacitor_SMD:C_0603_1608Metric_Pad1.08x0.95mm_HandSolder, F.Cu at (-4.68, 300.1)
- added C166: 10n, Capacitor_SMD:C_0603_1608Metric_Pad1.08x0.95mm_HandSolder, F.Cu at (-4.68, 302.6)
- added C167: 10n, Capacitor_SMD:C_0603_1608Metric_Pad1.08x0.95mm_HandSolder, F.Cu at (-4.68, 305.1)
- added C168: 2.2u, Capacitor_SMD:C_0603_1608Metric_Pad1.08x0.95mm_HandSolder, F.Cu at (-4.68, 307.6)
- added C169: 220p, Capacitor_SMD:C_0603_1608Metric_Pad1.08x0.95mm_HandSolder, F.Cu at (-4.68, 310.1)
- added C170: 1u, Capacitor_SMD:C_0603_1608Metric_Pad1.08x0.95mm_HandSolder, F.Cu at (-0.33, 287.5)
- added C171: 1u, Capacitor_SMD:C_0603_1608Metric_Pad1.08x0.95mm_HandSolder, F.Cu at (-0.33, 290.1)
- added C172: 220p, Capacitor_SMD:C_0603_1608Metric_Pad1.08x0.95mm_HandSolder, F.Cu at (-0.33, 292.6)
- added C173: 4.7u, Capacitor_SMD:C_0603_1608Metric_Pad1.08x0.95mm_HandSolder, F.Cu at (-0.33, 295.1)
- added C174: 100n, Capacitor_SMD:C_0603_1608Metric_Pad1.08x0.95mm_HandSolder, F.Cu at (-66.7, 313.2)
- added C20: C, Capacitor_SMD:C_0603_1608Metric_Pad1.08x0.95mm_HandSolder, F.Cu at (-93.4, 175.9)
- added C21: C, Capacitor_SMD:C_0603_1608Metric_Pad1.08x0.95mm_HandSolder, F.Cu at (-93.4, 178.4)
- added D4: D, Diode_THT:D_5W_P12.70mm_Horizontal, F.Cu at (-11.8, 328.0)
- added IC10: 551MLFT, Package_SO:SOIC-8_3.9x4.9mm_P1.27mm, F.Cu at (98.3, 125.7)
- added IC11: 551MLFT, Package_SO:SOIC-8_3.9x4.9mm_P1.27mm, F.Cu at (98.3, 132.2)
- added IC4: MC68901P, Package_DIP:DIP-48_W15.24mm_Socket, F.Cu at (-49.4, 210.7)
- added IC5: 551MLFT, Package_SO:SOIC-8_3.9x4.9mm_P1.27mm, F.Cu at (89.8, 125.7)
- added IC6: 501MLFT, Package_SO:SOIC-8_3.9x4.9mm_P1.27mm, F.Cu at (89.8, 132.2)
- added IC7: 551MLFT, Package_SO:SOIC-8_3.9x4.9mm_P1.27mm, F.Cu at (89.8, 138.6)
- added IC8: 551MLFT, Package_SO:SOIC-8_3.9x4.9mm_P1.27mm, F.Cu at (89.8, 145.1)
- added IC9: 501MLFT, Package_SO:SOIC-8_3.9x4.9mm_P1.27mm, F.Cu at (89.8, 151.5)
- added Q1: Q, RJK0651DPB-00:LFPAK_REN-M, F.Cu at (8.03, 318.4)
- added Q2: Q, RJK0651DPB-00:LFPAK_REN-M, F.Cu at (8.03, 325.5)
- added R42: R, Resistor_SMD:R_0603_1608Metric_Pad0.98x0.95mm_HandSolder, F.Cu at (-0.33, 302.6)
- added R43: 0, Resistor_SMD:R_0603_1608Metric_Pad0.98x0.95mm_HandSolder, F.Cu at (-0.33, 305.1)
- added R44: 2, Resistor_SMD:R_0603_1608Metric_Pad0.98x0.95mm_HandSolder, F.Cu at (-0.33, 307.6)
- added R45: 5m, Resistor_SMD:R_0603_1608Metric_Pad0.98x0.95mm_HandSolder, F.Cu at (-0.33, 310.1)
- added R46: 4m, Resistor_SMD:R_0603_1608Metric_Pad0.98x0.95mm_HandSolder, F.Cu at (4.02, 287.5)
- added R47: 4m, Resistor_SMD:R_0603_1608Metric_Pad0.98x0.95mm_HandSolder, F.Cu at (4.02, 290.1)
- added R48: 30, Resistor_SMD:R_0603_1608Metric_Pad0.98x0.95mm_HandSolder, F.Cu at (4.02, 292.6)
- added R49: 30, Resistor_SMD:R_0603_1608Metric_Pad0.98x0.95mm_HandSolder, F.Cu at (4.02, 295.1)
- added R50: 30, Resistor_SMD:R_0603_1608Metric_Pad0.98x0.95mm_HandSolder, F.Cu at (4.02, 297.6)
- added R51: 30, Resistor_SMD:R_0603_1608Metric_Pad0.98x0.95mm_HandSolder, F.Cu at (4.02, 300.1)
- added R52: 4.7, Resistor_SMD:R_0603_1608Metric_Pad0.98x0.95mm_HandSolder, F.Cu at (4.02, 302.6)
- added R53: 20k, Resistor_SMD:R_0603_1608Metric_Pad0.98x0.95mm_HandSolder, F.Cu at (4.02, 305.1)
- added R54: 20k, Resistor_SMD:R_0603_1608Metric_Pad0.98x0.95mm_HandSolder, F.Cu at (4.02, 307.6)
- added R55: 24.9k, Resistor_SMD:R_0603_1608Metric_Pad0.98x0.95mm_HandSolder, F.Cu at (4.02, 310.1)
- added R56: 30.1k, Resistor_SMD:R_0603_1608Metric_Pad0.98x0.95mm_HandSolder, F.Cu at (8.37, 287.5)
- added R57: 30.1k, Resistor_SMD:R_0603_1608Metric_Pad0.98x0.95mm_HandSolder, F.Cu at (8.37, 290.1)
- added R58: 17.8k, Resistor_SMD:R_0603_1608Metric_Pad0.98x0.95mm_HandSolder, F.Cu at (8.37, 292.6)
- added R59: 17.8k, Resistor_SMD:R_0603_1608Metric_Pad0.98x0.95mm_HandSolder, F.Cu at (8.37, 295.1)
- added R60: 11.3k, Resistor_SMD:R_0603_1608Metric_Pad0.98x0.95mm_HandSolder, F.Cu at (8.37, 297.6)
- added R61: 1.96k, Resistor_SMD:R_0603_1608Metric_Pad0.98x0.95mm_HandSolder, F.Cu at (8.37, 300.1)
- added R62: 1.96k, Resistor_SMD:R_0603_1608Metric_Pad0.98x0.95mm_HandSolder, F.Cu at (8.37, 302.6)
- added R63: 5k, Resistor_SMD:R_0603_1608Metric_Pad0.98x0.95mm_HandSolder, F.Cu at (8.37, 305.1)
- added R64: 10k, Resistor_SMD:R_0603_1608Metric_Pad0.98x0.95mm_HandSolder, F.Cu at (-66.7, 315.8)
- added R65: 1k, Resistor_SMD:R_0603_1608Metric_Pad0.98x0.95mm_HandSolder, F.Cu at (-66.7, 318.3)
- added R66: 1k, Resistor_SMD:R_0603_1608Metric_Pad0.98x0.95mm_HandSolder, F.Cu at (-66.7, 320.8)
- added R67: 1k, Resistor_SMD:R_0603_1608Metric_Pad0.98x0.95mm_HandSolder, F.Cu at (-66.7, 323.3)
- added RN1: 10k, Resistor_THT:R_Array_SIP8, F.Cu at (-90.8, 252.6)
- added RN2: 10k, Resistor_THT:R_Array_SIP5, F.Cu at (103.8, 316.8)
- added RN3: 330, Resistor_THT:R_Array_SIP4, F.Cu at (72.8, 158.3)
- added RN4: 1k, Resistor_THT:R_Array_SIP6, F.Cu at (53.7, 316.0)
- added U1: SIMM72 Slot A, Sockets:SIM72, F.Cu at (-74.1, 139.6)
- added U2: SIMM72 Slot B, Sockets:SIM72, F.Cu at (-74.1, 148.3)
- added U30: MAX1562ESA+, Package_SO:SOIC-8_3.9x4.9mm_P1.27mm, F.Cu at (102.9, 176.1)
- C1, C10, C11, C119, C12, C13, C14, C15, C16, C17, C2, C3, C4, C5, C54, C57, C6, C63, C66, C7, C71, C72, C73, C74, C75, C76, C79, C8, C80, C83, C84, C85, C9: footprint Capacitor_SMD:C_1206_3216Metric_Pad1.33x1.80mm_HandSolder -> Capacitor_SMD:C_0603_1608Metric_Pad1.08x0.95mm_HandSolder; moved to F.Cu
- C100, C106, C95: value 33p -> 1u; footprint Capacitor_SMD:C_1206_3216Metric_Pad1.33x1.80mm_HandSolder -> Capacitor_THT:CP_Radial_D5.0mm_P2.50mm
- C102: value 33p -> 100n; footprint Capacitor_SMD:C_1206_3216Metric_Pad1.33x1.80mm_HandSolder -> Capacitor_SMD:C_0603_1608Metric_Pad1.08x0.95mm_HandSolder
- C103, C115: value 47p -> 10u; footprint Capacitor_SMD:C_1206_3216Metric_Pad1.33x1.80mm_HandSolder -> Capacitor_THT:CP_Radial_D5.0mm_P2.50mm
- C104: value 1.2n -> 1u; footprint Capacitor_SMD:C_1206_3216Metric_Pad1.33x1.80mm_HandSolder -> Capacitor_SMD:C_0603_1608Metric_Pad1.08x0.95mm_HandSolder
- C105, C58, C59, C60, C61, C62: value 100n -> 1u; footprint Capacitor_SMD:C_1206_3216Metric_Pad1.33x1.80mm_HandSolder -> Capacitor_SMD:C_0603_1608Metric_Pad1.08x0.95mm_HandSolder; moved to F.Cu
- C107: value 100n -> 1u; footprint Capacitor_SMD:C_1206_3216Metric_Pad1.33x1.80mm_HandSolder -> Capacitor_THT:CP_Radial_D5.0mm_P2.50mm; moved to F.Cu
- C108: value 47p -> 470n; footprint Capacitor_SMD:C_1206_3216Metric_Pad1.33x1.80mm_HandSolder -> Capacitor_SMD:C_0603_1608Metric_Pad1.08x0.95mm_HandSolder
- C109: value 10u -> 33p; footprint Capacitor_THT:CP_Radial_D5.0mm_P2.50mm -> Capacitor_SMD:C_0603_1608Metric_Pad1.08x0.95mm_HandSolder
- C110: value 1.8n -> 1u; footprint Capacitor_SMD:C_1206_3216Metric_Pad1.33x1.80mm_HandSolder -> Capacitor_THT:CP_Radial_D5.0mm_P2.50mm
- C111: footprint Capacitor_SMD:C_1206_3216Metric_Pad1.33x1.80mm_HandSolder -> Capacitor_THT:CP_Radial_D5.0mm_P2.50mm
- C112, C130, C131, C132, C133, C88: footprint Capacitor_SMD:C_1206_3216Metric_Pad1.33x1.80mm_HandSolder -> Capacitor_SMD:C_0603_1608Metric_Pad1.08x0.95mm_HandSolder
- C113: value 10u -> 1u; footprint Capacitor_THT:CP_Radial_D5.0mm_P2.50mm -> Capacitor_SMD:C_0603_1608Metric_Pad1.08x0.95mm_HandSolder
- C114: value 1.8n -> 33p; footprint Capacitor_SMD:C_1206_3216Metric_Pad1.33x1.80mm_HandSolder -> Capacitor_SMD:C_0603_1608Metric_Pad1.08x0.95mm_HandSolder
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- renumbered H10 to H6, H11 to H7, H12 to H8, H13 to H9
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Connections:
- C1 pad 1: CPUPWR -> PWR_CPURAM
- C10 pad 2: CPUPWR -> PWR_CPURAM
- C100 pad 1: Net-(U20-XTAL1O) -> +5VA
- C100 pad 2: GND -> GNDA
- C102 pad 1: Net-(U20-XTAL2I) -> Net-(U26-VREFI)
- C102 pad 2: GND -> GNDA
- C103 pad 1: Net-(U19B--) -> Net-(U26-VREFI)
- C103 pad 2: Net-(C103-Pad2) -> GNDA
- C104 pad 1: Net-(U18B--) -> Net-(C104-Pad1)
- C104 pad 2: Net-(C104-Pad2) -> /Audio/LMIC
- C105 pad 1: +5VA -> Net-(C105-Pad1)
- C105 pad 2: GNDA -> /Audio/RLINE
- C106 pad 1: Net-(U20-XTAL2O) -> Net-(C106-Pad1)
- C106 pad 2: GND -> Net-(U24A-+)
- C107 pad 1: +5VA -> Net-(C107-Pad1)
- C107 pad 2: GNDA -> Net-(C107-Pad2)
- C108 pad 1: Net-(U21A--) -> GND
- C108 pad 2: Net-(C108-Pad2) -> Net-(U26-VREF)
- C109 pad 1: Net-(C109-Pad1) -> Net-(U26-XTAL1I)
- C109 pad 2: Net-(C109-Pad2) -> GND
- C11 pad 2: CPUPWR -> PWR_CPURAM
- C110 pad 1: Net-(C109-Pad1) -> Net-(C110-Pad1)
- C110 pad 2: GNDA -> Net-(U24B-+)
- C111 pad 1: Net-(U20-LFILT) -> Net-(C111-Pad1)
- C111 pad 2: GNDA -> Net-(C111-Pad2)
- C112 pad 1: Net-(U20-RFILT) -> Net-(C112-Pad1)
- C112 pad 2: GNDA -> /Audio/RMIC
- C113 pad 2: Net-(C113-Pad2) -> /Audio/LLINE
- C114 pad 1: Net-(C113-Pad1) -> Net-(U26-XTAL1O)
- C114 pad 2: GNDA -> GND
- C115 pad 1: Net-(U21B--) -> Net-(C115-Pad1)
- C115 pad 2: Net-(C115-Pad2) -> GNDA
- C116 pad 1: +12V -> Net-(U26-XTAL2I)
- C116 pad 2: -12V -> GND
- C117 pad 1: +3.3V -> Net-(U25B--)
- C117 pad 2: GND -> Net-(C113-Pad1)
- C118 pad 1: +3.3V -> Net-(U24B--)
- C118 pad 2: GND -> Net-(C112-Pad1)
- C119 pad 1: +3.3V -> +5VA
- C119 pad 2: GND -> GNDA
- C12 pad 1: CPUPWR -> PWR_CPURAM
- C120 pad 1: +5V -> Net-(U26-XTAL2O)
- C121 pad 1: Net-(J20-VBUS) -> +5VA
- C121 pad 2: GND -> GNDA
- C122 pad 1: /USB/X1 -> Net-(U27A--)
- C123 pad 2: GND -> Net-(C123-Pad2)
- C124 pad 1: Net-(C122-Pad2) -> Net-(C123-Pad1)
- C124 pad 2: GND -> GNDA
- C125 pad 1: Net-(U27-XA) -> Net-(U26-LFILT)
- C125 pad 2: GND -> GNDA
- C126 pad 1: GND -> Net-(U26-RFILT)
- C126 pad 2: Net-(U27-XB) -> GNDA
- C127 pad 1: +5V -> Net-(C127-Pad1)
- C127 pad 2: GND -> Net-(C127-Pad2)
- C128 pad 1: +5V -> Net-(C127-Pad1)
- C128 pad 2: GND -> GNDA
- C129 pad 1: +5V -> Net-(U27B--)
- C129 pad 2: GND -> Net-(C129-Pad2)
- C13 pad 1: CPUPWR -> PWR_CPURAM
- C130 pad 1: +5V -> +12V
- C130 pad 2: GND -> -12V
- C131 pad 1: +5V -> +3.3V
- C132 pad 1: +5V -> +3.3V
- C133 pad 1: +5V -> +3.3V
- C135 pad 1: +5V -> Net-(J18-VBUS)
- C136 pad 1: +5V -> /USB/X1
- C136 pad 2: GND -> Net-(C136-Pad2)
- C137 pad 1: +5V -> Net-(C137-Pad1)
- C138 pad 1: +5V -> Net-(C136-Pad2)
- C139 pad 1: +5V -> Net-(U31-CAP)
- C14 pad 1: CPUPWR -> PWR_CPURAM
- C140 pad 1: +5V -> +12V
- C141 pad 1: +5V -> PWR_CPURAM
- C148 pad 1: +5V -> +12V
- C149 pad 1: CPUPWR -> +5V
- C15 pad 2: CPUPWR -> PWR_CPURAM
- C16 pad 1: CPUPWR -> PWR_CPURAM
- C17 pad 1: CPUPWR -> PWR_CPURAM
- C18 pad 1: +5V -> PWR_FPGA
- C19 pad 1: CPUPWR -> PWR_FPGA
- C2 pad 1: CPUPWR -> PWR_CPURAM
- C22 pad 1: +12V -> PWR_FPGA
- C23 pad 1: +12V -> PWR_FPGA
- C24 pad 1: +5V -> PWR_FPGA
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
Commit message: Large changes: EHBCSimpleEmu, kicad, fwcode, docs
This commit contains some large changes:
- Removed EHBCSimpleEmu (Moved to kms1212/llemu, kms1212/qemu)
- (likely) Removed fwcode; now it only boots and stops
- Modified documents
Parts:
- removed BT1: Battery_Cell, Battery:BatteryHolder_ComfortableElectronic_CH273-2450_1x2450
- removed C100, C106, C107, C110, C111, C95, C96: 1u, Capacitor_THT:CP_Radial_D5.0mm_P2.50mm
- removed C101, C103, C115, C123, C127: 10u, Capacitor_THT:CP_Radial_D5.0mm_P2.50mm
- removed C102, C119, C121, C130, C131, C132, C133, C158, C162, C163, C174, C54, C57, C63, C66, C71, C72, C73, C74, C75, C76, C77, C78, C79, C80, C83, C84, C85, C86, C87, C88, C89, C90, C93, C94, C97, C98, C99: 100n, Capacitor_SMD:C_0603_1608Metric_Pad1.08x0.95mm_HandSolder
- removed C104, C105, C112, C113, C125, C126, C134, C159, C164, C165, C170, C171, C58, C59, C60, C61, C62: 1u, Capacitor_SMD:C_0603_1608Metric_Pad1.08x0.95mm_HandSolder
- removed C108: 470n, Capacitor_SMD:C_0603_1608Metric_Pad1.08x0.95mm_HandSolder
- removed C109, C114, C116, C120: 33p, Capacitor_SMD:C_0603_1608Metric_Pad1.08x0.95mm_HandSolder
- removed C117, C122, C129, C92: 47p, Capacitor_SMD:C_0603_1608Metric_Pad1.08x0.95mm_HandSolder
- removed C118, C91: 1.2n, Capacitor_SMD:C_0603_1608Metric_Pad1.08x0.95mm_HandSolder
- removed C124, C128: 1.8n, Capacitor_SMD:C_0603_1608Metric_Pad1.08x0.95mm_HandSolder
- removed C135, C173: 4.7u, Capacitor_SMD:C_0603_1608Metric_Pad1.08x0.95mm_HandSolder
- removed C136, C81, C82: 10p, Capacitor_SMD:C_0603_1608Metric_Pad1.08x0.95mm_HandSolder
- removed C137, C138, C55, C56, C69, C70: 22p, Capacitor_SMD:C_0603_1608Metric_Pad1.08x0.95mm_HandSolder
- removed C139: 47n, Capacitor_SMD:C_0603_1608Metric_Pad1.08x0.95mm_HandSolder
- removed C140, C29, C31, C32, C33, C34, C35, C36, C37, C38, C39, C40, C41, C42, C43, C44, C45, C46, C47, C48, C49, C50, C51, C52, C53: C, Capacitor_SMD:C_0603_1608Metric_Pad1.08x0.95mm_HandSolder
- removed C141, C142, C151, C152: 150u, Capacitor_THT:CP_Radial_D5.0mm_P2.50mm
- removed C143, C144, C145, C146, C153, C154, C155, C156: 22u, Capacitor_SMD:C_0603_1608Metric_Pad1.08x0.95mm_HandSolder
- removed C147, C149, C160: 470u, Capacitor_THT:CP_Radial_D8.0mm_P3.50mm
- removed C148, C150, C161: 47u, Capacitor_THT:CP_Radial_D8.0mm_P3.50mm
- removed C157: 10u, Capacitor_SMD:C_0603_1608Metric_Pad1.08x0.95mm_HandSolder
- removed C166, C167, C67, C68: 10n, Capacitor_SMD:C_0603_1608Metric_Pad1.08x0.95mm_HandSolder
- removed C168: 2.2u, Capacitor_SMD:C_0603_1608Metric_Pad1.08x0.95mm_HandSolder
- removed C169, C172: 220p, Capacitor_SMD:C_0603_1608Metric_Pad1.08x0.95mm_HandSolder
- removed C64, C65: 20p, Capacitor_SMD:C_0603_1608Metric_Pad1.08x0.95mm_HandSolder
- removed D1: LED, LED_THT:LED_D3.0mm
- removed D2, D3, D4: D, Diode_THT:D_5W_P12.70mm_Horizontal
- removed FB1: FerriteBead, Inductor_THT:L_Axial_L5.3mm_D2.2mm_P2.54mm_Vertical_Vishay_IM-1
- removed FB2, FB3: FerriteBead, Inductor_THT:L_Axial_L5.0mm_D3.6mm_P10.00mm_Horizontal_Murata_BL01RN1A2A2
- removed H1, H2, H3, H4, H5, H6, H7, H8, H9: M3_MH_Pad, MountingHole:MountingHole_3.2mm_M3_Pad
- removed IC10, IC11, IC5, IC7, IC8: 551MLFT, Package_SO:SOIC-8_3.9x4.9mm_P1.27mm
- removed IC4: MC68901P, Package_DIP:DIP-48_W15.24mm_Socket
- removed IC6, IC9: 501MLFT, Package_SO:SOIC-8_3.9x4.9mm_P1.27mm
- removed J14: RJ45_Amphenol_RJMG1BD3B8K1ANR, Connector_RJ:RJ45_Amphenol_RJMG1BD3B8K1ANR
- removed J15: IDC_PATA, Connector_IDC:IDC-Header_2x20_P2.54mm_Vertical
- removed J16: IDC_FDD, Connector_IDC:IDC-Header_2x17_P2.54mm_Vertical
- removed J17: STX-4335-5BGP-S1, STX43355BGPS1:STX43355BGPS1
- removed J18: USB_A, Connector_USB:USB_A_Wuerth_614004134726_Horizontal
- removed J19: ATX-24, Connector_Molex:Molex_Mini-Fit_Jr_5566-24A_2x12_P4.20mm_Vertical
- removed J20: ISP_SMC, Connector_PinSocket_2.54mm:PinSocket_2x03_P2.54mm_Vertical
- removed J21: ISP_FPGA, Connector_PinHeader_2.54mm:PinHeader_2x05_P2.54mm_Vertical
- removed L1, L2, L3, L4, L5, L6: L, Inductor_SMD:L_1206_3216Metric_Pad1.42x1.75mm_HandSolder
- removed L7: 2.2u, Inductor_SMD:L_1206_3216Metric_Pad1.42x1.75mm_HandSolder
- removed L8, L9: 4.7u, Inductor_SMD:L_10.4x10.4_H4.8
- removed Q1, Q2: Q, RJK0651DPB-00:LFPAK_REN-M
- removed R1, R2, R39, R4, R5, R64: 10k, Resistor_SMD:R_0603_1608Metric_Pad0.98x0.95mm_HandSolder
- removed R10, R44: 2, Resistor_SMD:R_0603_1608Metric_Pad0.98x0.95mm_HandSolder
- removed R11, R20: 1.5k, Resistor_SMD:R_0603_1608Metric_Pad0.98x0.95mm_HandSolder
- removed R12, R22: 11k, Resistor_SMD:R_0603_1608Metric_Pad0.98x0.95mm_HandSolder
- removed R13, R21: 22k, Resistor_SMD:R_0603_1608Metric_Pad0.98x0.95mm_HandSolder
- removed R14, R15, R17, R19: 47k, Resistor_SMD:R_0603_1608Metric_Pad0.98x0.95mm_HandSolder
- removed R16, R18: 5.1k, Resistor_SMD:R_0603_1608Metric_Pad0.98x0.95mm_HandSolder
- removed R23, R30: 18k, Resistor_SMD:R_0603_1608Metric_Pad0.98x0.95mm_HandSolder
- removed R24, R28: 680, Resistor_SMD:R_0603_1608Metric_Pad0.98x0.95mm_HandSolder
- removed R25, R29: 8.2k, Resistor_SMD:R_0603_1608Metric_Pad0.98x0.95mm_HandSolder
- removed R26, R27: 75, Resistor_SMD:R_0603_1608Metric_Pad0.98x0.95mm_HandSolder
- removed R3, R9: 330, Resistor_SMD:R_0603_1608Metric_Pad0.98x0.95mm_HandSolder
- removed R31, R32: 24, Resistor_SMD:R_0603_1608Metric_Pad0.98x0.95mm_HandSolder
- removed R33, R34: 15k, Resistor_SMD:R_0603_1608Metric_Pad0.98x0.95mm_HandSolder
- removed R35, R7: 1M, Resistor_SMD:R_0603_1608Metric_Pad0.98x0.95mm_HandSolder
- removed R36: 100, Resistor_SMD:R_0603_1608Metric_Pad0.98x0.95mm_HandSolder
- removed R37: 100k, Resistor_SMD:R_0603_1608Metric_Pad0.98x0.95mm_HandSolder
- removed R38: 470k, Resistor_SMD:R_0603_1608Metric_Pad0.98x0.95mm_HandSolder
- removed R40, R41, R42: R, Resistor_SMD:R_0603_1608Metric_Pad0.98x0.95mm_HandSolder
- removed R43: 0, Resistor_SMD:R_0603_1608Metric_Pad0.98x0.95mm_HandSolder
- removed R45: 5m, Resistor_SMD:R_0603_1608Metric_Pad0.98x0.95mm_HandSolder
- removed R46, R47: 4m, Resistor_SMD:R_0603_1608Metric_Pad0.98x0.95mm_HandSolder
- removed R48, R49, R50, R51: 30, Resistor_SMD:R_0603_1608Metric_Pad0.98x0.95mm_HandSolder
- removed R52: 4.7, Resistor_SMD:R_0603_1608Metric_Pad0.98x0.95mm_HandSolder
- removed R53, R54: 20k, Resistor_SMD:R_0603_1608Metric_Pad0.98x0.95mm_HandSolder
- removed R55: 24.9k, Resistor_SMD:R_0603_1608Metric_Pad0.98x0.95mm_HandSolder
- removed R56, R57: 30.1k, Resistor_SMD:R_0603_1608Metric_Pad0.98x0.95mm_HandSolder
- removed R58, R59: 17.8k, Resistor_SMD:R_0603_1608Metric_Pad0.98x0.95mm_HandSolder
- removed R6: 200, Resistor_SMD:R_0603_1608Metric_Pad0.98x0.95mm_HandSolder
- removed R60: 11.3k, Resistor_SMD:R_0603_1608Metric_Pad0.98x0.95mm_HandSolder
- removed R61, R62: 1.96k, Resistor_SMD:R_0603_1608Metric_Pad0.98x0.95mm_HandSolder
- removed R63: 5k, Resistor_SMD:R_0603_1608Metric_Pad0.98x0.95mm_HandSolder
- removed R65, R66, R67: 1k, Resistor_SMD:R_0603_1608Metric_Pad0.98x0.95mm_HandSolder
- removed R8: 27k, Resistor_SMD:R_0603_1608Metric_Pad0.98x0.95mm_HandSolder
- removed RN1: 10k, Resistor_THT:R_Array_SIP8
- removed RN2: 10k, Resistor_THT:R_Array_SIP5
- removed RN3: 330, Resistor_THT:R_Array_SIP4
- removed RN4: 1k, Resistor_THT:R_Array_SIP6
- removed RN5: 10k, Resistor_THT:R_Array_SIP9
- removed RN6: 1k, Resistor_THT:R_Array_SIP5
- removed TP1: TestPoint_2Pole, Connector_PinHeader_1.00mm:PinHeader_1x02_P1.00mm_Vertical
- removed U26: CS4231A, Package_LCC:PLCC-68_THT-Socket
- removed U29: USB6B1, Package_SO:SOIC-8_3.9x4.9mm_P1.27mm
- removed U30: MAX1562ESA+, Package_SO:SOIC-8_3.9x4.9mm_P1.27mm
- removed U31: MX8315MC, Package_SO:SOIC-14_3.9x8.7mm_P1.27mm
- removed U32: DS1307+, Package_DIP:DIP-8_W7.62mm_Socket
- removed U33: ICS542, Package_SO:SOIC-8_3.9x4.9mm_P1.27mm
- removed U34: PAC1953x-x4MX, Package_DFN_QFN:VQFN-16-1EP_3x3mm_P0.5mm_EP1.1x1.1mm
- removed U35, U36: 0651, RJK0651DPB-00:LFPAK_REN
- removed U37: LTC3886, Package_DFN_QFN:Linear_UGK52_QFN-46-52
- removed U38, U39: 0653, RJK0651DPB-00:LFPAK_REN
- removed U40: AT17LV010A, Package_DIP:DIP-8_W7.62mm
- removed X1: 14.31818M, Oscillator:Oscillator_SMD_SeikoEpson_SG8002CA-4Pin_7.0x5.0mm
- removed X2: 70M, Oscillator:Oscillator_SMD_SeikoEpson_SG8002CA-4Pin_7.0x5.0mm
- removed Y1: 16M, Crystal:Crystal_HC52-6mm_Vertical
- removed Y2: 8M, Crystal:Crystal_HC52-6mm_Vertical
- removed Y3: 20M, Crystal:Crystal_HC52-6mm_Vertical
- removed Y4: 24M, Crystal:Crystal_HC52-6mm_Vertical
- removed Y5: 24.576M, Crystal:Crystal_HC52-6mm_Vertical
- removed Y6: 16.9344M, Crystal:Crystal_HC52-6mm_Vertical
- removed Y7: 48M, Crystal:Crystal_HC52-6mm_Vertical
- removed Y8: 32.768k, Crystal:Crystal_Round_D2.0mm_Vertical
- C1, C10, C11, C12, C13, C14, C15, C16, C17, C2, C3, C4, C5, C6, C7, C8, C9: moved to B.Cu
- C18, C19, C20, C21, C22, C23, C24, C25, C26, C27, C28, C30: value C -> 100n; footprint Capacitor_SMD:C_0603_1608Metric_Pad1.08x0.95mm_HandSolder -> Capacitor_THT:C_Disc_D6.0mm_W2.5mm_P5.00mm
- IC1: value MC68881FN -> MC68030RC; footprint Package_LCC:PLCC-68_THT-Socket -> m68k-hbc-ic:PGA128
- IC2: value MC68030RC -> MC68881FN; footprint m68k-hbc-ic:PGA128 -> Package_LCC:PLCC-68_THT-Socket
- IC3: value 23LCV1024-I_SN -> MC68901P; footprint Package_SO:SOIC-8_3.9x4.9mm_P1.27mm -> Package_DIP:DIP-48_W15.24mm_Socket
- J1: value SIMM80_Cache -> PEP_Data_DIN41612_3x32; footprint 5822030-4:58220304 -> m68k-hbc-conn:PEP_Board
- J10: value ICSP_SMC -> USB_A; footprint Connector_PinSocket_2.54mm:PinSocket_2x03_P2.54mm_Vertical -> Connector_USB:USB_A_Wuerth_614004134726_Horizontal
- J11: value Conn_02x08_Odd_Even -> RJ45_Bel_SI-60062-F; footprint Connector_PinHeader_2.54mm:PinHeader_2x08_P2.54mm_Vertical -> Connector_RJ:RJ45_Bel_SI-60062-F
- J12: value 5747840-4 -> ATX-24; footprint 57478404:57478404 -> Connector_Molex:Molex_Mini-Fit_Jr_5566-24A_2x12_P4.20mm_Vertical
- J13: value KMDGX-6SG_P-S4N -> SIMM80_Cache; footprint KMDGX6SGPS4N:KMDGX6SGPS4N -> 5822030-4:58220304
- J2: value PEP_Power_DIN41612_3x10 -> PEP_Data_DIN41612_3x32; footprint Connector_DIN:DIN41612_C3_3x10_Female_Vertical_THT -> m68k-hbc-conn:PEP_Board
- J3, J4: value PEP_Power_DIN41612_3x10 -> Bus_ISA_16bit; footprint Connector_DIN:DIN41612_C3_3x10_Female_Vertical_THT -> Sockets:ISA_16bit
- J5: value PEP_Data_DIN41612_3x32 -> IDC_PATA; footprint Connector_DIN:DIN41612_C_3x32_Female_Vertical_THT -> Connector_IDC:IDC-Header_2x20_P2.54mm_Vertical
- J6: value PEP_Data_DIN41612_3x32 -> IDC_FDD; footprint Connector_DIN:DIN41612_C_3x32_Female_Vertical_THT -> Connector_IDC:IDC-Header_2x17_P2.54mm_Vertical
- J7: value PEP_Data_DIN41612_3x32 -> 5747840-4; footprint Connector_DIN:DIN41612_C_3x32_Female_Vertical_THT -> 57478404:57478404
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Connections:
- net IRQ_USBC renamed /Bus/MMIO/Ethernet/~{DTACK}
- C1 pad 1: PWR_CPURAM -> +5VCPU
- C10 pad 1: GND -> +5VCPU
- C10 pad 2: PWR_CPURAM -> GND
- C11 pad 1: GND -> +5VCPU
- C11 pad 2: PWR_CPURAM -> GND
- C12 pad 1: PWR_CPURAM -> +5VCPU
- C13 pad 1: PWR_CPURAM -> +5VCPU
- C14 pad 1: PWR_CPURAM -> +5VCPU
- C15 pad 1: GND -> +5VCPU
- C15 pad 2: PWR_CPURAM -> GND
- C16 pad 1: PWR_CPURAM -> +5VCPU
- C17 pad 1: PWR_CPURAM -> +5VCPU
- C18 pad 1: PWR_FPGA -> +5VCPU
- C19 pad 1: PWR_FPGA -> +5VCPU
- C2 pad 1: PWR_CPURAM -> +5VCPU
- C20 pad 1: PWR_FPGA -> +5VPER
- C21 pad 1: PWR_FPGA -> +5VPER
- C22 pad 1: PWR_FPGA -> +5VPER
- C23 pad 1: PWR_FPGA -> +5VPER
- C24 pad 1: PWR_FPGA -> +5VPER
- C25 pad 1: PWR_FPGA -> +5VPER
- C26 pad 1: PWR_FPGA -> +5VPER
- C27 pad 1: PWR_FPGA -> +5VPER
- C28 pad 1: PWR_FPGA -> +5VPER
- C3 pad 1: GND -> +5VCPU
- C3 pad 2: PWR_CPURAM -> GND
- C30 pad 1: PWR_FPGA -> +5VPER
- C4 pad 1: PWR_CPURAM -> +5VCPU
- C5 pad 1: GND -> +5VCPU
- C5 pad 2: PWR_CPURAM -> GND
- C6 pad 1: PWR_CPURAM -> +5VCPU
- C7 pad 1: PWR_CPURAM -> +5VCPU
- C8 pad 1: PWR_CPURAM -> +5VCPU
- C9 pad 1: PWR_CPURAM -> +5VCPU
- IC3 pad 1: ~{CS_NVRAM} -> /Bus/MMIO/Serial/R/~{W}
- IC3 pad 2: /FWMEM/SYS_MISO -> /Bus/A0
- IC3 pad 3: unconnected-(IC3-NC-Pad3) -> /Bus/A1
- IC3 pad 4: GND -> /Bus/A2
- IC3 pad 5: /FWMEM/SYS_MOSI -> /Bus/A3
- IC3 pad 6: /FWMEM/SYS_SCK -> /Bus/A4
- IC3 pad 7: +BATT -> unconnected-(IC3A-TC-Pad7)
- IC3 pad 8: PWR_CPURAM -> unconnected-(IC3A-SO-Pad8)
- J10 pad 1: /SMC/SMC_MISO -> unconnected-(J10-VBUS-Pad1)
- J10 pad 2: Net-(J10-Pin_2) -> unconnected-(J10-D--Pad2)
- J10 pad 3: /SMC/SMC_SCK -> unconnected-(J10-D+-Pad3)
- J10 pad 4: /SMC/SMC_MOSI -> unconnected-(J10-GND-Pad4)
- J10 pad 5: ~{RST_SMC} -> unconnected-(J10-Shield-Pad5)
- J11 pad 1: GND -> Net-(J11-TD+)
- J11 pad 2: BUZ -> Net-(J11-TCT)
- J11 pad 3: SMC_TX -> Net-(J11-TD-)
- J11 pad 4: unconnected-(J11-Pin_4-Pad4) -> Net-(J11-RD+)
- J11 pad 5: SMC_RX -> Net-(J11-RCT)
- J11 pad 6: unconnected-(J11-Pin_6-Pad6) -> Net-(J11-RD-)
- J11 pad 7: GND -> (no net)
- J12 pad 1: unconnected-(J12-Pad1) -> +3.3V
- J12 pad 2: Net-(U17-T1OUT) -> +3.3V
- J12 pad 3: Net-(U17-R1IN) -> GND
- J12 pad 4: unconnected-(J12-Pad4) -> +5V
- J12 pad 6: unconnected-(J12-Pad6) -> +5V
- J12 pad 7: unconnected-(J12-Pad7) -> GND
- J12 pad 9: unconnected-(J12-Pad9) -> +5VSB
- J13 pad MH1: GNDPWR -> (no net)
- J13 pad MH2: GNDPWR -> (no net)
- J13 pad MH3: GNDPWR -> (no net)
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Routing:
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- added copper zone on B.Cu, net GND
- added copper zone on F.Cu, net GND
Other:
- board text removed: "68k30 HBC Motherboard"
- board text removed: "ATX-Size 12inx9.6in"
- board text removed: "Designed by kms1212(Minsu Kwon)"
- board text removed: "Rev.1 2023/xx/xx"
