File: kicad/projects/videocard/videocard.kicad_pcb (KiCad board)
At the start: 4 copper layers, 218.4 x 106.7 mm, 62 parts, among them J1 DE15_Receptacle_HighDensity_M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, J2 PEP_Data_DIN41612_3x32, J3 PEP_Power_DIN41612_3x10, U1 SSD1963QL9, U10 TXB0108DQSR, U11 PCA9306D, U12 CY7C1041D, U13 CY7C1041D, U14 CY7C1041D, U15 CY7C1041D, U16 AD1580BRTZ-REEL7, U17 74LS137, U18 TXB0108DQSR, U19 74LS573, U2 TXB0108DQSR, U20 74LS245, U21 74LS573, U22 74LS573, U23 74LS245, U3 CY7C1041D, U4 CY7C1041D, U5 CY7C1041D, U6 CY7C1041D, U7 TXB0108DQSR, U8 MC68000FN, U9 ADV7123

Commit message: Some Updates
Parts:
- removed R2: 1k, Resistor_THT:R_Axial_DIN0204_L3.6mm_D1.6mm_P5.08mm_Horizontal
- removed R3: 530, Resistor_THT:R_Axial_DIN0204_L3.6mm_D1.6mm_P5.08mm_Horizontal
- removed U13, U14, U15: CY7C1041D, Package_SO:TSOP-II-44_10.16x18.41mm_P0.8mm
- removed U16: AD1580BRTZ-REEL7, SOT96P237X112-3N:SOT96P237X112-3N
- removed U17: 74LS137, Package_DIP:DIP-16_W7.62mm_Socket
- removed U18: TXB0108DQSR, Package_SON:USON-20_2x4mm_P0.4mm
- removed U19, U21, U22: 74LS573, Package_DIP:DIP-20_W7.62mm_Socket
- removed U20, U23: 74LS245, Package_DIP:DIP-20_W7.62mm_Socket
- added C33: 100n, Capacitor_SMD:C_0603_1608Metric_Pad1.08x0.95mm_HandSolder, F.Cu at (217.2, 103.5)
- added C34: 100n, Capacitor_SMD:C_0603_1608Metric_Pad1.08x0.95mm_HandSolder, F.Cu at (210.8, 103.5)
- added C35: 100n, Capacitor_SMD:C_0603_1608Metric_Pad1.08x0.95mm_HandSolder, F.Cu at (203.2, 114.7)
- added C36: 100n, Capacitor_SMD:C_0603_1608Metric_Pad1.08x0.95mm_HandSolder, F.Cu at (203.2, 121.3)
- added C37: 100n, Capacitor_SMD:C_0603_1608Metric_Pad1.08x0.95mm_HandSolder, F.Cu at (203.2, 131.2)
- added C38: 100n, Capacitor_SMD:C_0603_1608Metric_Pad1.08x0.95mm_HandSolder, F.Cu at (162.6, 99.9)
- added C39: 10n, Capacitor_SMD:C_0603_1608Metric_Pad1.08x0.95mm_HandSolder, F.Cu at (164.5, 99.9)
- added C40: 100n, Capacitor_SMD:C_0603_1608Metric_Pad1.08x0.95mm_HandSolder, F.Cu at (162.6, 96.5)
- added C41: 10n, Capacitor_SMD:C_0603_1608Metric_Pad1.08x0.95mm_HandSolder, F.Cu at (164.5, 96.5)
- added C42: 100n, Capacitor_SMD:C_0603_1608Metric_Pad1.08x0.95mm_HandSolder, F.Cu at (175.3, 95.7)
- added C43: 10n, Capacitor_SMD:C_0603_1608Metric_Pad1.08x0.95mm_HandSolder, F.Cu at (177.2, 95.7)
- added J4: DE15_Receptacle_HighDensity_MountingHoles, Connector_Dsub:DSUB-15-HD_Female_Horizontal_P2.29x1.98mm_EdgePinOffset3.03mm_Housed_MountingHolesOffset4.94mm, F.Cu at (153.8, 105.2)
- added J6: Conn_01x40_MountingPin, Connector_FFC-FPC:TE_4-1734839-0_1x40-1MP_P0.5mm_Horizontal, F.Cu at (186.4, 99.7)
- added R5: 1k, Resistor_SMD:R_0603_1608Metric_Pad0.98x0.95mm_HandSolder, F.Cu at (166.9, 112.8)
- added R6: 560, Resistor_SMD:R_0603_1608Metric_Pad0.98x0.95mm_HandSolder, F.Cu at (166.0, 108.0)
- added R7: 200k, Resistor_SMD:R_0603_1608Metric_Pad0.98x0.95mm_HandSolder, F.Cu at (162.6, 85.7)
- added RN2: 75, Resistor_THT:R_Array_SIP4, F.Cu at (159.4, 108.0)
- added RN3: 10k, Resistor_THT:R_Array_SIP4, F.Cu at (254.6, 102.9)
- added SW1: SW_SPST, Button_Switch_SMD:SW_Push_1P1T_NO_6x6mm_H9.5mm, F.Cu at (219.1, 90.8)
- added SW2: SW_DIP_x04, Package_DIP:DIP-8_W7.62mm, F.Cu at (272.4, 92.7)
- C1, C11, C12, C13, C14, C15, C16, C17, C20, C23, C24, C25, C26, C28, C3, C30, C31, C32, C4, C5, C6, C7, C8: footprint Capacitor_SMD:C_1206_3216Metric_Pad1.33x1.80mm_HandSolder -> Capacitor_SMD:C_0603_1608Metric_Pad1.08x0.95mm_HandSolder
- C10, C22, C9: value 1u -> 100n; footprint Capacitor_SMD:C_1206_3216Metric_Pad1.33x1.80mm_HandSolder -> Capacitor_SMD:C_0603_1608Metric_Pad1.08x0.95mm_HandSolder
- C18, C19: value 100n -> 200n; footprint Capacitor_SMD:C_1206_3216Metric_Pad1.33x1.80mm_HandSolder -> Capacitor_SMD:C_0603_1608Metric_Pad1.08x0.95mm_HandSolder
- C2, C21: value 100n -> 1u; footprint Capacitor_SMD:C_1206_3216Metric_Pad1.33x1.80mm_HandSolder -> Capacitor_SMD:C_0603_1608Metric_Pad1.08x0.95mm_HandSolder
- C27: value 10n -> 100n; footprint Capacitor_SMD:C_1206_3216Metric_Pad1.33x1.80mm_HandSolder -> Capacitor_SMD:C_0603_1608Metric_Pad1.08x0.95mm_HandSolder
- C29: value 100n -> 4.7u; footprint Capacitor_SMD:C_1206_3216Metric_Pad1.33x1.80mm_HandSolder -> Capacitor_THT:CP_Radial_D5.0mm_P2.50mm
- J1: value DE15_Receptacle_HighDensity_MountingHoles -> Conn_ARM_JTAG_SWD_20; footprint Connector_Dsub:DSUB-15-HD_Female_Horizontal_P2.29x1.98mm_EdgePinOffset3.03mm_Housed_MountingHolesOffset4.94mm -> Connector_IDC:IDC-Header_2x10_P2.54mm_Vertical
- J2: value PEP_Data_DIN41612_3x32 -> PEP_Power_DIN41612_3x10; footprint Connector_DIN:DIN41612_C_3x32_Male_Horizontal_THT -> Connector_DIN:DIN41612_C3_3x10_Male_Horizontal_THT
- J3: value PEP_Power_DIN41612_3x10 -> PEP_Data_DIN41612_3x32; footprint Connector_DIN:DIN41612_C3_3x10_Male_Horizontal_THT -> Connector_DIN:DIN41612_C_3x32_Male_Horizontal_THT
- R1: value 200k -> 10k; footprint Resistor_THT:R_Axial_DIN0204_L3.6mm_D1.6mm_P5.08mm_Horizontal -> Resistor_SMD:R_0603_1608Metric_Pad0.98x0.95mm_HandSolder
- RN1: value 75 -> 10k
- U1: value SSD1963QL9 -> MT48LC16M16A2P; footprint Package_QFP:LQFP-128_14x14mm_P0.4mm -> Package_SO:TSOP-II-54_22.2x10.16mm_P0.8mm
- U10: value TXB0108DQSR -> TXS0108EPW; footprint Package_SON:USON-20_2x4mm_P0.4mm -> Package_SO:TSSOP-20_4.4x6.5mm_P0.65mm
- U11: value PCA9306D -> TXS0108EPW; footprint Package_SO:SO-8_3.9x4.9mm_P1.27mm -> Package_SO:TSSOP-20_4.4x6.5mm_P0.65mm
- U12: value CY7C1041D -> PCA9306D; footprint Package_SO:TSOP-II-44_10.16x18.41mm_P0.8mm -> Package_SO:SO-8_3.9x4.9mm_P1.27mm
- U2: value TXB0108DQSR -> MT48LC16M16A2P; footprint Package_SON:USON-20_2x4mm_P0.4mm -> Package_SO:TSOP-II-54_22.2x10.16mm_P0.8mm
- U3, U6: value CY7C1041D -> 74ALVC164245DGG,51; footprint Package_SO:TSOP-II-44_10.16x18.41mm_P0.8mm -> Package_SO:TSSOP-48_8x12.5mm_P0.5mm
- U4: value CY7C1041D -> STM32H743BITx; footprint Package_SO:TSOP-II-44_10.16x18.41mm_P0.8mm -> Package_QFP:LQFP-208_28x28mm_P0.5mm
- U5: value CY7C1041D -> ADV7123; footprint Package_SO:TSOP-II-44_10.16x18.41mm_P0.8mm -> Package_QFP:LQFP-48_7x7mm_P0.5mm
- U7: value TXB0108DQSR -> AD1580BRTZ-REEL7; footprint Package_SON:USON-20_2x4mm_P0.4mm -> Package_TO_SOT_SMD:SOT-23-3
- U8: value MC68000FN -> 74LVC2T45DC; footprint Package_LCC:PLCC-68_THT-Socket -> Package_SO:VSSOP-8_2.3x2mm_P0.5mm
- U9: value ADV7123 -> PCA9306D; footprint Package_QFP:LQFP-48_7x7mm_P0.5mm -> Package_SO:SO-8_3.9x4.9mm_P1.27mm
- moved C20 162.2 mm to (164.5, 103.7), turned to 90 degrees
- moved RN1 126.4 mm to (285.1, 102.9)
- moved U5 123.8 mm to (170.8, 101.4), turned to 180 degrees
- moved C29 123.7 mm to (296.0, 149.2), turned to 0 degrees
- moved C18 115.6 mm to (210.8, 101.6)
- moved U11 109.8 mm to (261.0, 149.9), turned to -90 degrees
- moved U6 98.5 mm to (233.0, 149.9), turned to 90 degrees
- moved C19 86.4 mm to (239.4, 113.0), turned to 90 degrees
- moved J1 86.3 mm to (239.4, 97.2), turned to 90 degrees
- moved C26 84.9 mm to (237.5, 129.9), turned to 90 degrees
- moved C11 83.5 mm to (271.8, 106.7)
- moved U3 82.0 mm to (214.0, 149.9), turned to 90 degrees
- moved C27 81.2 mm to (237.5, 123.8), turned to 90 degrees
- moved C10 79.4 mm to (261.0, 123.8), turned to 90 degrees
- moved C9 77.6 mm to (261.0, 116.4), turned to 90 degrees
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Connections:
- C1 pad 1: +5V -> GND
- C1 pad 2: GND -> /~{RST}
- C12 pad 1: +1V2 -> +3.3V
- C13 pad 1: +5V -> +3.3V
- C15 pad 1: +5V -> +3.3V
- C17 pad 1: +5V -> +3.3V
- C18 pad 1: +5V -> Net-(C18-Pad1)
- C19 pad 1: +5V -> Net-(C18-Pad1)
- C2 pad 2: GND -> Net-(U4-VREF+)
- C20 pad 1: +5V -> Net-(U5-COMP)
- C20 pad 2: GND -> +3.3V
- C21 pad 1: Net-(U9-COMP) -> Net-(U5-Vref)
- C21 pad 2: +3.3VA -> GNDA
- C22 pad 1: Net-(U16-V+) -> +3.3V
- C22 pad 2: GNDA -> GND
- C23 pad 1: +5V -> +3.3V
- C24 pad 1: +5V -> +3.3V
- C26 pad 1: +3.3VA -> +3.3V
- C26 pad 2: GNDA -> GND
- C27 pad 1: +3.3VA -> +3.3V
- C27 pad 2: GNDA -> GND
- C28 pad 1: GND -> +3.3V
- C28 pad 2: +5V -> GND
- C29 pad 1: GND -> +3.3V
- C29 pad 2: +5V -> GND
- C3 pad 1: +5V -> +3.3V
- C3 pad 2: GND -> Net-(U4-VREF+)
- C30 pad 1: GND -> +3.3V
- C30 pad 2: +5V -> GND
- C31 pad 1: GND -> +3.3V
- C31 pad 2: +5V -> GND
- C32 pad 1: GND -> +3.3V
- C32 pad 2: +5V -> GND
- C4 pad 1: +5V -> +3.3V
- C5 pad 1: +5V -> +3.3V
- C6 pad 1: +5V -> +3.3V
- C7 pad 1: +5V -> +3.3V
- C8 pad 1: +5V -> +3.3V
- C9 pad 1: +1V2 -> +3.3V
- J1 pad 1: /RAO -> +3.3V
- J1 pad 11: unconnected-(J1-Pad11) -> Net-(J1-RTCK)
- J1 pad 12: /DDCSDA -> GND
- J1 pad 13: /HSYNC -> /TDO
- J1 pad 14: /VSYNC -> GND
- J1 pad 15: /DDCSCL -> /~{SRST}
- J1 pad 2: /GAO -> +3.3V
- J1 pad 3: /BAO -> /~{TRST}
- J1 pad 4: unconnected-(J1-Pad4) -> GND
- J1 pad 5: GND -> /TDI
- J1 pad 6: GNDA -> GND
- J1 pad 7: GNDA -> /TMS
- J1 pad 8: GNDA -> GND
- J1 pad 9: unconnected-(J1-Pad9) -> /TCK
- J2 pad a10: /PR/~{W} -> GND
- J2 pad a2: GND -> +12V
- J2 pad a3: unconnected-(J2-~{IACK}-Pada3) -> +12V
- J2 pad a4: unconnected-(J2-~{IRQ}-Pada4) -> +5VP
- J2 pad a5: GND -> +5V
- J2 pad a6: /PSIZ1 -> +5V
- J2 pad a7: /PSIZ0 -> +5V
- J2 pad a8: /~{PDSACK1} -> +3.3V
- J2 pad a9: /~{PDSACK0} -> +3.3V
- J2 pad b10: /PA16 -> GND
- J2 pad b2: GND -> +12V
- J2 pad b3: unconnected-(J2-~{PEACK}-Padb3) -> +12V
- J2 pad b4: unconnected-(J2-~{PERR}-Padb4) -> -12V
- J2 pad b6: /PA20 -> GND
- J2 pad b7: /PA21 -> +5V
- J2 pad b8: /PA22 -> +3.3V
- J2 pad b9: /PA23 -> +3.3V
- J2 pad c10: /PD14 -> GND
- J2 pad c2: unconnected-(J2-CLK_10MHz-Padc2) -> +12V
- J2 pad c3: unconnected-(J2-~{CRST}-Padc3) -> +12V
- J2 pad c4: /SDA -> -5V
- J2 pad c5: /SCL -> +5V
- J2 pad c6: unconnected-(J2-NC-Padc6) -> +5V
- J2 pad c7: unconnected-(J2-NC-Padc7) -> +5V
- J2 pad c8: GND -> +3.3V
- J2 pad c9: /PD15 -> +3.3V
- J3 pad a10: GND -> /P_OP0
- J3 pad a2: +12V -> GND
- J3 pad a3: +12V -> unconnected-(J3-~{IACK}-Pada3)
- J3 pad a4: +5VP -> /~{P_IRQ}
- J3 pad a5: +5V -> GND
- J3 pad a6: +5V -> /~{P_INIT}
- J3 pad a7: +5V -> /P_OP3
- J3 pad a8: +3.3V -> /P_OP2
- J3 pad a9: +3.3V -> /P_OP1
- J3 pad b10: GND -> unconnected-(J3-A16-Padb10)
- J3 pad b2: +12V -> GND
- J3 pad b3: +12V -> /~{P_CERR}
- J3 pad b4: -12V -> /~{P_PERR}
- J3 pad b6: GND -> unconnected-(J3-A20-Padb6)
- J3 pad b7: +5V -> unconnected-(J3-A21-Padb7)
- J3 pad b8: +3.3V -> unconnected-(J3-A22-Padb8)
- J3 pad b9: +3.3V -> unconnected-(J3-A23-Padb9)
- J3 pad c10: GND -> /P_AD30
- J3 pad c2: +12V -> unconnected-(J3-CLK10M-Padc2)
- J3 pad c3: +12V -> /~{P_RST}
- J3 pad c4: -5V -> /P_SDA
- J3 pad c5: +5V -> /P_SCL
- J3 pad c6: +5V -> unconnected-(J3-APAR1-Padc6)
- J3 pad c7: +5V -> unconnected-(J3-APAR0-Padc7)
- J3 pad c8: +3.3V -> GND
- J3 pad c9: +3.3V -> /P_AD31
- R1 pad 1: +5V -> +3.3V
- R1 pad 2: Net-(U11-EN) -> /~{RST}
- RN1 pad 1: GNDA -> GND
- RN1 pad 2: /RAO -> /BOOT0
- RN1 pad 3: /GAO -> /~{PSAVE}
- RN1 pad 4: /BAO -> /PDR_ON
- U1 pad 1: +1V2 -> +3.3V
- U1 pad 10: /33D3 -> /SDQ5
- U1 pad 11: /33D4 -> /SDQ6
- U1 pad 12: +3.3V -> GND
- U1 pad 13: GND -> /SDQ7
- U1 pad 14: +1V2 -> +3.3V
- U1 pad 15: unconnected-(U1A-CLK-Pad15) -> /NBL0
- U1 pad 16: +3.3V -> /~{SDWE}
- U1 pad 17: GND -> /~{SDCAS}
- U1 pad 18: +1V2 -> /~{SDRAS}
- U1 pad 19: GND -> /~{SDEN0}
- U1 pad 2: GND -> /SDQ0
- U1 pad 20: GND -> /BA0
- U1 pad 21: +1V2 -> /BA1
- U1 pad 22: unconnected-(U1A-XTAL_IN-Pad22) -> /DRA10
- U1 pad 23: GND -> /DRA0
- U1 pad 24: unconnected-(U1A-XTAL_OUT-Pad24) -> /DRA1
- U1 pad 25: +1V2 -> /DRA2
- U1 pad 26: GND -> /DRA3
- U1 pad 28: /R7 -> GND
- U1 pad 29: /R6 -> /DRA4
- U1 pad 3: GND -> +3.3V
- U1 pad 30: /R5 -> /DRA5
- U1 pad 31: /R4 -> /DRA6
- U1 pad 32: +1V2 -> /DRA7
- U1 pad 33: GND -> /DRA8
- U1 pad 34: +3.3V -> /DRA9
- U1 pad 35: /R1 -> /DRA11
- U1 pad 36: /~{PSAVE} -> /DRA12
- U1 pad 37: /33DDCSCL -> /SDCKE0
- U1 pad 38: /33DDCSDA -> /SDCLK
- U1 pad 39: unconnected-(U1A-GPIO3-Pad39) -> /NBL1
- U1 pad 4: +3.3V -> /SDQ1
- U1 pad 40: +1V2 -> unconnected-(U1-NC-Pad40)
- U1 pad 42: +3.3V -> /SDQ8
- U1 pad 43: /33VSYNC -> +3.3V
- U1 pad 44: /33HSYNC -> /SDQ9
- U1 pad 45: /PXCLK -> /SDQ10
- U1 pad 46: +1V2 -> GND
- U1 pad 47: GND -> /SDQ11
- U1 pad 48: +3.3V -> /SDQ12
- U1 pad 49: /~{BLANK} -> +3.3V
- U1 pad 5: GND -> /SDQ2
- U1 pad 50: unconnected-(U1A-TE-Pad50) -> /SDQ13
- U1 pad 51: unconnected-(U1A-PWM-Pad51) -> /SDQ14
- U1 pad 52: unconnected-(U1A-GAMAS0-Pad52) -> GND
- U1 pad 53: unconnected-(U1A-GAMAS1-Pad53) -> /SDQ15
- U1 pad 54: +3.3V -> GND
- U1 pad 6: +1V2 -> GND
- U1 pad 7: /33D0 -> /SDQ3
- U1 pad 8: /33D1 -> /SDQ4
- U1 pad 9: /33D2 -> +3.3V
- U10 pad 1: /33A1 -> /PARITY
- U10 pad 12: unconnected-(U10-B7-Pad12) -> /~{P_DS}
- U10 pad 13: unconnected-(U10-B6-Pad13) -> /~{P_DACK}
- U10 pad 14: unconnected-(U10-B5-Pad14) -> /~{P_MRDY}
- U10 pad 15: GND -> /~{P_CRDY}
- U10 pad 16: +5V -> /~{P_CEN}
- U10 pad 17: unconnected-(U10-B4-Pad17) -> /~{P_CERR}
- U10 pad 18: /R/~{W} -> /~{P_PERR}
- U10 pad 19: /E -> unconnected-(U10-VCCB-Pad19)
- U10 pad 2: /33E -> unconnected-(U10-VCCA-Pad2)
- U10 pad 20: /A1 -> /P_PARITY
- U10 pad 3: /33R/~{W} -> /~{PERR}
- U10 pad 4: unconnected-(U10-A4-Pad4) -> /~{CERR}
- U10 pad 5: +3.3V -> /~{CEN}
- U10 pad 6: unconnected-(U10-OE-Pad6) -> /~{CRDY}
- U10 pad 7: unconnected-(U10-A5-Pad7) -> /~{MRDY}
- U10 pad 8: unconnected-(U10-A6-Pad8) -> /~{DACK}
- U10 pad 9: unconnected-(U10-A7-Pad9) -> /~{DS}
- U11 pad 1: GND -> /OP0
- U11 pad 2: +3.3V -> unconnected-(U11-VCCA-Pad2)
- U11 pad 3: /33DDCSCL -> /OP1
- U11 pad 4: /33DDCSDA -> /OP2
- U11 pad 5: /DDCSDA -> /OP3
- U11 pad 6: /DDCSCL -> /~{STOP}
- U11 pad 7: Net-(U11-EN) -> /~{RST}
- U11 pad 8: Net-(U11-EN) -> /~{IRQ}
- U12 pad 1: /A1 -> unconnected-(U12-GND-Pad1)
- U12 pad 2: /A2 -> unconnected-(U12-VREF1-Pad2)
- U12 pad 3: /A3 -> /SCL
- U12 pad 4: /A4 -> /SDA
- U12 pad 5: /A5 -> /P_SDA
- U12 pad 6: ~{RAMCS4} -> /P_SCL
- U12 pad 7: /D0 -> unconnected-(U12-VREF2-Pad7)
- U12 pad 8: /D1 -> unconnected-(U12-EN-Pad8)
- U2 pad 1: /33D0 -> +3.3V
- U2 pad 10: /33D7 -> /SDQ5
- U2 pad 11: /D7 -> /SDQ6
- U2 pad 12: /D6 -> GND
- U2 pad 13: /D5 -> /SDQ7
- U2 pad 14: /D4 -> +3.3V
- U2 pad 15: GND -> /NBL0
- U2 pad 16: +5V -> /~{SDWE}
- U2 pad 17: /D3 -> /~{SDCAS}
- U2 pad 18: /D2 -> /~{SDRAS}
- U2 pad 19: /D1 -> /~{SDEN1}
- U2 pad 2: /33D1 -> /SDQ0
- U2 pad 20: /D0 -> /BA0
- U2 pad 3: /33D2 -> +3.3V
- U2 pad 4: /33D3 -> /SDQ1
- U2 pad 5: +3.3V -> /SDQ2
- U2 pad 6: unconnected-(U2-OE-Pad6) -> GND
- U2 pad 7: /33D4 -> /SDQ3
- U2 pad 8: /33D5 -> /SDQ4
- U2 pad 9: /33D6 -> +3.3V
- U3 pad 1: /A1 -> unconnected-(U3-1DIR-Pad1)
- U3 pad 10: /D3 -> unconnected-(U3-GND-Pad10)
- U3 pad 11: +5V -> /P_AD6
- U3 pad 12: GND -> /P_AD7
- U3 pad 13: /D4 -> /P_AD8
- U3 pad 14: /D5 -> /P_AD9
- U3 pad 15: /D6 -> unconnected-(U3-GND_5-Pad15)
- U3 pad 16: /D7 -> /P_AD10
- U3 pad 17: unconnected-(U3-~{WE}-Pad17) -> /P_AD11
- U3 pad 18: /A6 -> unconnected-(U3-VCC(B)-Pad18)
- U3 pad 19: /A7 -> /P_AD12
- U3 pad 2: /A2 -> /P_AD0
- U3 pad 20: /A8 -> /P_AD13
- U3 pad 21: /A9 -> unconnected-(U3-GND_7-Pad21)
- U3 pad 22: /A10 -> /P_AD14
- U3 pad 23: /A11 -> /P_AD15
- U3 pad 24: /A12 -> unconnected-(U3-2DIR-Pad24)
- U3 pad 25: /A13 -> unconnected-(U3-~2OE-Pad25)
- U3 pad 26: /A14 -> /AD15
- U3 pad 27: /A15 -> /AD14
- U3 pad 29: /D8 -> /AD13
- U3 pad 3: /A3 -> /P_AD1
- U3 pad 30: /D9 -> /AD12
- U3 pad 31: /D10 -> unconnected-(U3-VCC(A)_2-Pad31)
- U3 pad 32: /D11 -> /AD11
- U3 pad 33: +5V -> /AD10
- U3 pad 34: GND -> unconnected-(U3-GND_4-Pad34)
- U3 pad 35: /D12 -> /AD9
- U3 pad 36: /D13 -> /AD8
- U3 pad 37: /D14 -> /AD7
- U3 pad 38: /D15 -> /AD6
- U3 pad 39: /~{LDS} -> unconnected-(U3-GND_8-Pad39)
- U3 pad 4: /A4 -> unconnected-(U3-GND_3-Pad4)
- U3 pad 40: /~{UDS} -> /AD5
- U3 pad 41: unconnected-(U3-~{OE}-Pad41) -> /AD4
- U3 pad 42: /A16 -> unconnected-(U3-VCC(A)-Pad42)
- U3 pad 43: /A17 -> /AD3
- U3 pad 44: /A18 -> /AD2
- U3 pad 5: /A5 -> /P_AD2
- U3 pad 6: ~{RAMCS0} -> /P_AD3
- U3 pad 7: /D0 -> unconnected-(U3-VCC(B)_2-Pad7)
- U3 pad 8: /D1 -> /P_AD4
- U3 pad 9: /D2 -> /P_AD5
- U4 pad 1: /A1 -> unconnected-(U4-PE2-Pad1)
- U4 pad 10: /D3 -> unconnected-(U4-PC15-Pad10)
- U4 pad 11: +5V -> /DISP_VSYNC
- U4 pad 12: GND -> /DISP_HSYNC
- U4 pad 13: /D4 -> /DISP_G6
- U4 pad 14: /D5 -> GND
- U4 pad 15: /D6 -> +3.3V
- U4 pad 16: /D7 -> /DRA0
- U4 pad 17: unconnected-(U4-~{WE}-Pad17) -> /DRA1
- U4 pad 18: /A6 -> /DRA2
- U4 pad 19: /A7 -> unconnected-(U4-PI12-Pad19)
- U4 pad 2: /A2 -> unconnected-(U4-PE3-Pad2)
- U4 pad 20: /A8 -> unconnected-(U4-PI13-Pad20)
- U4 pad 21: /A9 -> /DISP_PCLK
- U4 pad 22: /A10 -> /DRA3
- U4 pad 23: /A11 -> /DRA4
- U4 pad 24: /A12 -> /DRA5
- U4 pad 25: /A13 -> GND
- U4 pad 26: /A14 -> +3.3V
- U4 pad 27: /A15 -> unconnected-(U4-PF6-Pad27)
- U4 pad 29: /D8 -> unconnected-(U4-PF8-Pad29)
- U4 pad 3: /A3 -> /DISP_B0
- U4 pad 30: /D9 -> unconnected-(U4-PF9-Pad30)
- U4 pad 31: /D10 -> /DISP_DE
- U4 pad 32: /D11 -> OSC_HSE
- U4 pad 33: +5V -> unconnected-(U4-PH1-Pad33)
- U4 pad 34: GND -> /~{RST}
- U4 pad 35: /D12 -> /~{SDWE}
- U4 pad 36: /D13 -> unconnected-(U4-PC1-Pad36)
- U4 pad 37: /D14 -> /~{SDEN0}
- U4 pad 38: /D15 -> /SDCKE0
- U4 pad 39: /~{LDS} -> +3.3V
- U4 pad 4: /A4 -> /DISP_G0
- U4 pad 40: /~{UDS} -> GND
- U4 pad 41: unconnected-(U4-~{OE}-Pad41) -> Net-(U4-VREF+)
- U4 pad 42: /A16 -> +3.3V
- U4 pad 43: /A17 -> unconnected-(U4-PA0-Pad43)
- U4 pad 44: /A18 -> /DISP_R2
- U4 pad 5: /A5 -> /DISP_G1
- U4 pad 6: ~{RAMCS1} -> +3.3V
- U4 pad 7: /D0 -> unconnected-(U4-PI8-Pad7)
- U4 pad 8: /D1 -> /~{MRDY}
- U4 pad 9: /D2 -> unconnected-(U4-PC14-Pad9)
- U5 pad 1: /A1 -> GND
- U5 pad 10: /D3 -> /DISP_G7
- U5 pad 11: +5V -> /DISP_DE
- U5 pad 13: /D4 -> +3.3V
- U5 pad 14: /D5 -> GND
- U5 pad 15: /D6 -> GND
- U5 pad 16: /D7 -> /DISP_B0
- U5 pad 17: unconnected-(U5-~{WE}-Pad17) -> /DISP_B1
- U5 pad 18: /A6 -> /DISP_B2
- U5 pad 19: /A7 -> /DISP_B3
- U5 pad 2: /A2 -> GND
- U5 pad 20: /A8 -> /DISP_B4
- U5 pad 21: /A9 -> /DISP_B5
- U5 pad 22: /A10 -> /DISP_B6
- U5 pad 23: /A11 -> /DISP_B7
- U5 pad 24: /A12 -> /DISP_PCLK
- U5 pad 25: /A13 -> GNDA
- U5 pad 26: /A14 -> GNDA
- U5 pad 27: /A15 -> GNDA
- U5 pad 29: /D8 -> +3.3V
- U5 pad 3: /A3 -> /DISP_G0
- U5 pad 30: /D9 -> +3.3V
- U5 pad 31: /D10 -> GNDA
- U5 pad 32: /D11 -> /GREEN
- U5 pad 33: +5V -> GNDA
- U5 pad 34: GND -> /RED
- U5 pad 35: /D12 -> Net-(U5-COMP)
- U5 pad 36: /D13 -> Net-(U5-Vref)
- U5 pad 37: /D14 -> Net-(U5-Rset)
- U5 pad 38: /D15 -> /~{PSAVE}
- U5 pad 39: /~{LDS} -> GND
- U5 pad 4: /A4 -> /DISP_G1
- U5 pad 40: /~{UDS} -> GND
- U5 pad 41: unconnected-(U5-~{OE}-Pad41) -> /DISP_R0
- U5 pad 42: /A16 -> /DISP_R1
- U5 pad 43: /A17 -> /DISP_R2
- U5 pad 44: /A18 -> /DISP_R3
- U5 pad 5: /A5 -> /DISP_G2
- U5 pad 6: ~{RAMCS2} -> /DISP_G3
- U5 pad 7: /D0 -> /DISP_G4
- U5 pad 8: /D1 -> /DISP_G5
- U5 pad 9: /D2 -> /DISP_G6
- U6 pad 1: /A1 -> unconnected-(U6-1DIR-Pad1)
- U6 pad 10: /D3 -> unconnected-(U6-GND-Pad10)
- U6 pad 11: +5V -> /P_AD22
- U6 pad 12: GND -> /P_AD23
- U6 pad 13: /D4 -> /P_AD24
- U6 pad 14: /D5 -> /P_AD25
- U6 pad 15: /D6 -> unconnected-(U6-GND_5-Pad15)
- U6 pad 16: /D7 -> /P_AD26
- U6 pad 17: unconnected-(U6-~{WE}-Pad17) -> /P_AD27
- U6 pad 18: /A6 -> unconnected-(U6-VCC(B)-Pad18)
- U6 pad 19: /A7 -> /P_AD28
- U6 pad 2: /A2 -> /P_AD16
- U6 pad 20: /A8 -> /P_AD29
- U6 pad 21: /A9 -> unconnected-(U6-GND_7-Pad21)
- U6 pad 22: /A10 -> /P_AD30
- U6 pad 23: /A11 -> /P_AD31
- U6 pad 24: /A12 -> unconnected-(U6-2DIR-Pad24)
- U6 pad 25: /A13 -> unconnected-(U6-~2OE-Pad25)
- U6 pad 26: /A14 -> /AD31
- U6 pad 27: /A15 -> /AD30
- U6 pad 29: /D8 -> /AD29
- U6 pad 3: /A3 -> /P_AD17
- U6 pad 30: /D9 -> /AD28
- U6 pad 31: /D10 -> unconnected-(U6-VCC(A)_2-Pad31)
- U6 pad 32: /D11 -> /AD27
- U6 pad 33: +5V -> /AD26
- U6 pad 34: GND -> unconnected-(U6-GND_4-Pad34)
- U6 pad 35: /D12 -> /AD25
- U6 pad 36: /D13 -> /AD24
- U6 pad 37: /D14 -> /AD23
- U6 pad 38: /D15 -> /AD22
- U6 pad 39: /~{LDS} -> unconnected-(U6-GND_8-Pad39)
- U6 pad 4: /A4 -> unconnected-(U6-GND_3-Pad4)
- U6 pad 40: /~{UDS} -> /AD21
- U6 pad 41: unconnected-(U6-~{OE}-Pad41) -> /AD20
- U6 pad 42: /A16 -> unconnected-(U6-VCC(A)-Pad42)
- U6 pad 43: /A17 -> /AD19
- U6 pad 44: /A18 -> /AD18
- U6 pad 5: /A5 -> /P_AD18
- U6 pad 6: ~{RAMCS3} -> /P_AD19
- U6 pad 7: /D0 -> unconnected-(U6-VCC(B)_2-Pad7)
- U6 pad 8: /D1 -> /P_AD20
- U6 pad 9: /D2 -> /P_AD21
- U7 pad 1: /33D8 -> Net-(U5-Vref)
- U7 pad 2: /33D9 -> GNDA
- U7 pad 3: /33D10 -> unconnected-(U7-NC-Pad3)
- U8 pad 1: /D4 -> +3.3V
- U8 pad 2: /D3 -> /DISP_VSYNC
- U8 pad 3: /D2 -> /DISP_HSYNC
- U8 pad 4: /D1 -> GND
- U8 pad 5: /D0 -> +3.3V
- U8 pad 6: /~{AS} -> /HSYNC
- U8 pad 7: /~{UDS} -> /VSYNC
- U8 pad 8: /~{LDS} -> +5V
- U9 pad 2: GND -> +3.3V
- U9 pad 3: /G0 -> /DISP_SCL
- U9 pad 4: /G1 -> /DISP_SDA
- U9 pad 5: /G2 -> /DDC_SDA
- U9 pad 6: /G3 -> /DDC_SCL
- U9 pad 7: /G4 -> +5V
- U9 pad 8: /G5 -> Net-(U9-EN)
Other:
- board size 218.4 x 106.7 mm -> 181.6 x 105.4 mm
