File: kicad/projects/videocard/videocard.kicad_sch (KiCad schematic)
At the start: 55 parts, among them J1 DE15_Receptacle_HighDensity_M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, J2 PEP_Data_DIN41612_3x32, J3 PEP_Power_DIN41612_3x10, U1 SSD1963QL9, U10 TXB0108DQSR, U11 PCA9306D, U12 CY7C1041D, U13 CY7C1041D, U14 CY7C1041D, U15 CY7C1041D, U16 AD1580BRTZ-REEL7, U17 EPM7128SLC84-15, U18 TXB0108DQSR, U19 74LS137, U2 TXB0108DQSR, U20 74LS139, U21 74LS348, U3 CY7C1041D, U4 CY7C1041D, U5 CY7C1041D, U6 CY7C1041D, U7 TXB0108DQSR, U8 MC68000FN, U9 ADV7123

Commit message: Some Updates
Parts:
- removed C1, C11, C12, C13, C14, C15, C16, C17, C18, C19, C2, C20, C21, C24, C25, C26, C3, C4, C5, C6, C7, C8: 100n, Capacitor_SMD:C_1206_3216Metric_Pad1.33x1.80mm_HandSolder, symbol Device:C
- removed C10, C22, C9: 1u, Capacitor_SMD:C_1206_3216Metric_Pad1.33x1.80mm_HandSolder, symbol Device:C
- removed C23: 100n, Capacitor_THT:C_Disc_D3.0mm_W1.6mm_P2.50mm, symbol Device:C
- removed C27: 10n, Capacitor_SMD:C_1206_3216Metric_Pad1.33x1.80mm_HandSolder, symbol Device:C
- removed J1: DE15_Receptacle_HighDensity_MountingHoles, Connector_Dsub:DSUB-15-HD_Female_Horizontal_P2.29x1.98mm_EdgePinOffset3.03mm_Housed_MountingHolesOffset4.94mm, symbol Connector:DE15_Receptacle_HighDensity_MountingHoles
- removed J2: PEP_Data_DIN41612_3x32, Connector_DIN:DIN41612_C_3x32_Female_Vertical_THT, symbol EPBus:PEP_Data_DIN41612_3x32
- removed J3: PEP_Power_DIN41612_3x10, Connector_DIN:DIN41612_C3_3x10_Male_Horizontal_THT, symbol EPBus:PEP_Power_DIN41612_3x10
- removed R1: 200k, Resistor_THT:R_Axial_DIN0204_L3.6mm_D1.6mm_P5.08mm_Horizontal, symbol Device:R
- removed R2: 1k, Resistor_THT:R_Axial_DIN0204_L3.6mm_D1.6mm_P5.08mm_Horizontal, symbol Device:R
- removed R3: 530, Resistor_THT:R_Axial_DIN0204_L3.6mm_D1.6mm_P5.08mm_Horizontal, symbol Device:R
- removed RN1: 75, Resistor_THT:R_Array_SIP4, symbol Device:R_Network03
- removed U1: SSD1963QL9, Package_QFP:LQFP-128_14x14mm_P0.4mm, symbol SSD1963QL9:SSD1963QL9
- removed U10, U18, U2, U7: TXB0108DQSR, Package_SON:USON-20_2x4mm_P0.4mm, symbol Logic_LevelTranslator:TXB0108DQSR
- removed U11: PCA9306D, Package_SO:SO-8_3.9x4.9mm_P1.27mm, symbol Interface:PCA9306D
- removed U12, U13, U14, U15, U3, U4, U5, U6: CY7C1041D, Package_SO:TSOP-II-44_10.16x18.41mm_P0.8mm, symbol CY7C1041D:CY7C1041D
- removed U16: AD1580BRTZ-REEL7, SOT96P237X112-3N:SOT96P237X112-3N, symbol AD1580BRTZ-REEL7:AD1580BRTZ-REEL7
- removed U17: EPM7128SLC84-15, Package_LCC:PLCC-84, symbol EPM7128SLC84-15:EPM7128SLC84-15
- removed U19: 74LS137, Package_DIP:DIP-16_W7.62mm_Socket, symbol 74xx:74LS137
- removed U20: 74LS139, symbol 74xx:74LS139
- removed U21: 74LS348, symbol 74xx:74LS348
- removed U8: MC68000FN, Package_LCC:PLCC-68_THT-Socket, symbol CPU_NXP_68000:MC68000FN
- removed U9: ADV7123, Package_QFP:LQFP-48_7x7mm_P0.5mm, symbol analog_devices:ADV7123
- added J2: PEP_Power_DIN41612_3x10, Connector_DIN:DIN41612_C3_3x10_Male_Horizontal_THT, symbol m68k-hbc-conn:PEP_Power_DIN41612_3x10
- added J3: PEP_Data_DIN41612_3x32, Connector_DIN:DIN41612_C_3x32_Female_Vertical_THT, symbol m68k-hbc-conn:PEP_Data_DIN41612_3x32
- added U1: EPF6016QC240, Package_QFP:PQFP-240_32.1x32.1mm_P0.5mm, symbol m68k-hbc-ic:EPF6016QC240
- added U2: TMS34020APCM, symbol m68k-hbc-ic:TMS34020APCM
Connections:
- net +12V: now also J2.a2 (+12V), J2.a3 (+12V), J2.b2 (+12V), J2.b3 (+12V), J2.c2 (+12V), J2.c3 (+12V)
- net +3.3V: now also J2.a8 (+3.3V), J2.a9 (+3.3V), J2.b8 (+3.3V), J2.b9 (+3.3V), J2.c8 (+3.3V), J2.c9 (+3.3V)
- net +5V: now also J2.a5 (+5V), J2.a6 (+5V), J2.a7 (+5V), J2.b7 (+5V), J2.c5 (+5V), J2.c6 (+5V), J2.c7 (+5V)
- net +5VP: now also J2.a4 (+5VSB)
- net -12V: now also J2.b4 (-12V)
- net -5V: now also J2.c4 (-5V)
- net GND: now also J2.a1 (GND), J2.a10 (GND), J2.b1 (GND), J2.b10 (GND), J2.b5 (GND), J2.b6 (~{PRES}), J2.c1 (GND), J2.c10 (GND), J3.a1 (GND), J3.a14 (GND), J3.a2 (~{PRES}), J3.a23 (GND), J3.a3 (GND), J3.a32 (GND), J3.b1 (GND), J3.b10 (GND), J3.b11 (GND), J3.b12 (GND), J3.b13 (GND), J3.b14 (GND), J3.b15 (GND), J3.b16 (GND), J3.b17 (GND), J3.b18 (GND), J3.b19 (GND), J3.b2 (GND), J3.b20 (GND), J3.b21 (GND), J3.b22 (GND), J3.b23 (GND), J3.b24 (GND), J3.b25 (GND), J3.b26 (GND), J3.b27 (GND), J3.b28 (GND), J3.b29 (GND), J3.b3 (GND), J3.b30 (GND), J3.b31 (GND), J3.b32 (GND), J3.b4 (GND), J3.b5 (GND), J3.b6 (GND), J3.b7 (GND), J3.b8 (GND), J3.b9 (GND), J3.c1 (GND), J3.c17 (GND), J3.c25 (GND), J3.c26 (GND), J3.c27 (GND), J3.c30 (GND), J3.c32 (GND), J3.c6 (GND), J3.c7 (GND), J3.c8 (GND)
- new net HA0: U1.84 (IO)
- new net HA1: U1.85 (IO)
- new net HA10: U1.98 (IO), U2.41 (HA10)
- new net HA11: U1.99 (IO), U2.40 (HA11)
- new net HA12: U1.100 (IO), U2.39 (HA12)
- new net HA13: U1.101 (IO), U2.38 (HA13)
- new net HA14: U1.102 (IO), U2.37 (HA14)
- new net HA15: U1.103 (IO), U2.36 (HA15)
- new net HA16: U1.104 (IO), U2.35 (HA16)
- new net HA17: U1.105 (IO), U2.33 (HA17)
- new net HA18: U1.106 (IO), U2.32 (HA18)
- new net HA19: U1.107 (IO), U2.31 (HA19)
- new net HA2: U1.86 (IO)
- new net HA20: U1.108 (IO), U2.30 (HA20)
- new net HA21: U1.111 (IO), U2.29 (HA21)
- new net HA22: U1.112 (IO), U2.28 (HA22)
- new net HA23: U1.113 (IO), U2.27 (HA23)
- new net HA24: U1.114 (IO), U2.26 (HA24)
- new net HA25: U1.115 (IO), U2.25 (HA25)
- new net HA26: U1.116 (IO), U2.24 (HA26)
- new net HA27: U1.118 (IO), U2.23 (HA27)
- new net HA28: U1.119 (IO), U2.22 (HA28)
- new net HA29: U1.121 (IO), U2.21 (HA29)
- new net HA3: U1.87 (IO)
- new net HA30: U1.122 (IO), U2.20 (HA30)
- new net HA31: U1.123 (IO), U2.19 (HA31)
- new net HA4: U1.88 (IO)
- new net HA5: U1.93 (IO), U2.46 (HA5)
- new net HA6: U1.94 (IO), U2.45 (HA6)
- new net HA7: U1.95 (IO), U2.44 (HA7)
- new net HA8: U1.96 (IO), U2.43 (HA8)
- new net HA9: U1.97 (IO), U2.42 (HA9)
- new net HD0: U1.125 (IO)
- new net HD1: U1.126 (IO)
- new net HD10: U1.138 (IO)
- new net HD11: U1.139 (IO)
- new net HD12: U1.140 (IO)
- new net HD13: U1.141 (IO)
- new net HD14: U1.142 (IO)
- new net HD15: U1.143 (IO)
- new net HD16: U1.144 (IO)
- new net HD17: U1.145 (IO)
- new net HD18: U1.146 (IO)
- new net HD19: U1.147 (IO)
- new net HD2: U1.127 (IO)
- new net HD20: U1.153 (IO)
- new net HD21: U1.154 (IO)
- new net HD22: U1.156 (IO)
- new net HD23: U1.157 (IO)
- new net HD24: U1.158 (IO)
- new net HD25: U1.159 (IO)
- new net HD26: U1.160 (IO)
- new net HD27: U1.162 (IO)
- new net HD28: U1.163 (IO)
- new net HD29: U1.164 (IO)
- new net HD3: U1.128 (IO)
- new net HD30: U1.165 (IO)
- new net HD31: U1.167 (IO)
- new net HD4: U1.132 (IO)
- new net HD5: U1.133 (IO)
- new net HD6: U1.134 (IO)
- new net HD7: U1.135 (IO)
- new net HD8: U1.136 (IO)
- new net HD9: U1.137 (IO)
- new net P_AD0: J3.a31 (AD0), U1.1 (IO)
- new net P_AD1: J3.a30 (AD1), U1.2 (IO)
- new net P_AD10: J3.a20 (AD10), U1.15 (IO)
- new net P_AD11: J3.a19 (AD11), U1.16 (IO)
- new net P_AD12: J3.a18 (AD12), U1.17 (IO)
- new net P_AD13: J3.a17 (AD13), U1.18 (IO)
- new net P_AD14: J3.a16 (AD14), U1.19 (IO)
- new net P_AD15: J3.a15 (AD15), U1.20 (IO)
- new net P_AD16: J3.c25 (GND), U1.21 (IO)
- new net P_AD17: J3.c24 (AD17), U1.23 (IO)
- new net P_AD18: J3.c23 (AD18), U1.24 (IO)
- new net P_AD19: J3.c22 (AD19), U1.25 (IO)
- new net P_AD2: J3.a29 (AD2), U1.3 (IO)
- new net P_AD20: J3.c21 (AD20), U1.26 (IO)
- new net P_AD21: J3.c20 (AD21), U1.27 (IO)
- new net P_AD22: J3.c19 (AD22), U1.33 (IO)
- new net P_AD23: J3.c18 (AD23), U1.34 (IO)
- new net P_AD24: J3.c16 (AD24), U1.35 (IO)
- new net P_AD25: J3.c15 (AD25), U1.36 (IO)
- new net P_AD26: J3.c14 (AD26), U1.37 (IO)
- new net P_AD27: J3.c13 (AD27), U1.38 (IO)
- new net P_AD28: J3.c12 (AD28), U1.39 (IO)
- new net P_AD29: J3.c11 (AD29), U1.40 (IO)
- new net P_AD3: J3.a28 (AD3), U1.4 (IO)
- new net P_AD30: J3.c10 (AD30), U1.41 (IO)
- new net P_AD31: J3.c9 (AD31), U1.42 (IO)
- new net P_AD4: J3.a27 (AD4), U1.5 (IO)
- new net P_AD5: J3.a26 (AD5), U1.6 (IO)
- new net P_AD6: J3.a25 (AD6), U1.7 (IO)
- new net P_AD7: J3.a24 (AD7), U1.8 (IO)
- new net P_AD8: J3.a22 (AD8), U1.13 (IO)
- new net P_AD9: J3.a21 (AD9), U1.14 (IO)
- new net P_CLK: J3.c2 (CLK), U1.66 (IO)
- new net P_OP0: J3.a10 (OP0), U1.48 (IO)
- new net P_OP1: J3.a9 (OP1), U1.53 (IO)
- new net P_OP2: J3.a8 (OP2), U1.55 (IO)
- new net P_OP3: J3.a7 (OP3), U1.56 (IO)
- new net P_PARITY: J3.c31 (PAR), U1.43 (IO)
- new net P_SCL: J3.c5 (I2CSCL), U1.63 (IO)
- new net P_SDA: J3.c4 (I2CSDA), U1.64 (IO)
- new net ~{P_CEN}: J3.a13 (~{EN}), U1.45 (IO)
- new net ~{P_CERR}: J3.c29 (~{PERR}), U1.62 (IO)
- new net ~{P_CRDY}: J3.a12 (~{CRDY}), U1.46 (IO)
- new net ~{P_INIT}: J3.a6 (~{INIT}), U1.57 (IO)
- new net ~{P_IRQ}: J3.a4 (~{IRQ}), U1.59 (IO)
- new net ~{P_MRDY}: J3.a11 (~{MRDY}), U1.47 (IO)
- new net ~{P_PERR}: J3.c28 (~{CERR}), U1.60 (IO)
- new net ~{P_RST}: J3.c3 (~{RST}), U1.65 (IO)
- new net ~{P_STOP}: J3.a5 (~{STOP}), U1.58 (IO)
- no-connect marks 7 -> 0
